File: flagship/drive-io.kicad_sch (KiCad schematic)
At the start: 11 parts, among them J4 DRIVE_COMMS, J5 DRIVE_MOTION, U10 74AHCT125, U9 THVD1450

Commit message: flagship: motor-switch note carries the measured 150 uF drive-side capacitance and the pre-charge numbers
Co-Authored-By: Claude Opus 5.5 (1M context) <noreply@anthropic.com>
Parts:
- removed J4: DRIVE_COMMS, symbol Connector_Generic:Conn_01x08
- removed J5: DRIVE_MOTION, symbol Connector_Generic:Conn_01x04
- removed R17, R18, R19: 10k, Resistor_SMD:R_0805_2012Metric, symbol Device:R
- removed R20, R21, R22: 1k, Resistor_SMD:R_0805_2012Metric, symbol Device:R
- removed R23: 120R_DNP, Resistor_SMD:R_0805_2012Metric, symbol Device:R
- removed U10: 74AHCT125, flagship:TSSOP-14_L5.0-W4.4-P0.65-LS6.4-BL, symbol flagship:SN74AHCT125PWR
- removed U9: THVD1450, flagship:SOIC-8_L4.9-W3.9-P1.27-LS6.0-BL, symbol flagship:THVD1450DR
Other:
- note removed: "DRIVE IO (record sections 11-12; SPEC rulings: 3.3 V RS485 non-isolated, quadrature via 74AHCT125, JST GH signals). Connectors are generic placeholders: operator picks parts and pin order. U9 THVD1450 from a P4 UART in RS485 half-duplex mode; DE and /RE tied, one GPIO. R23 termination fitted-not-populated (short point-to-point run). U10: 3.3 V GPIO in (TTL thresholds), 5 V out to the drive's opto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"

Commit message: flagship: schematic skeleton across all seven sheets
Candidate ICs placed with cross-sheet nets as global labels and a design note per sheet
citing the record: LTC4364IS-2 input protection with INA228 Kelvin shunt and mirrored bulk;
TPS48111 back-to-back motor switch with pre-charge, MOTOR_EN pulldown, INA ALERT hardware
cut; TLV1805 + TLV431 self-acting regen clamp, 2x TO-263, external connector and
parallel/replace jumper; 3x TPS54560B bucks (12/5/3.3 V); Stamp-P4 with fixed pins only
(GPIO assignment follows layout, per ruling); THVD1450 RS485, 74AHCT125 quadrature, drive
status inputs; INA228, thermistor and fan headers. Connectors are generic placeholders.

SPEC.md: rulings for no RP2350 (P4 LP-core emits quadrature) and passive sizes.
Libraries normalized to ASCII (LCSC Chinese manufacturer names, en-dash pin name) after
they broke the MCP server's Windows-codepage reads.

ERC: 109 unconnected pins (detailing), 62 pin-type warnings (LCSC symbols ship
unspecified pin types), 13 one-sided labels (GPIO pending layout); 0 dangling.

Co-Authored-By: Claude Opus 5.5 (1M context) <noreply@anthropic.com>
Parts:
- added J4: DRIVE_COMMS, symbol Connector_Generic:Conn_01x08
- added J5: DRIVE_MOTION, symbol Connector_Generic:Conn_01x04
- added R17, R18, R19: 10k, Resistor_SMD:R_0805_2012Metric, symbol Device:R
- added R20, R21, R22: 1k, Resistor_SMD:R_0805_2012Metric, symbol Device:R
- added R23: 120R_DNP, Resistor_SMD:R_0805_2012Metric, symbol Device:R
- added U10: 74AHCT125, flagship:TSSOP-14_L5.0-W4.4-P0.65-LS6.4-BL, symbol flagship:SN74AHCT125PWR
- added U9: THVD1450, flagship:SOIC-8_L4.9-W3.9-P1.27-LS6.0-BL, symbol flagship:THVD1450DR
Connections:
- new net +3V3: R17.1, R18.1, R19.1, U9.8 (VCC)
- new net +5V: J4.1 (Pin_1), U10.10 (~{3OE}), U10.13 (~{4OE}), U10.14 (VCC)
- new net DRV_485A: J4.3 (Pin_3), R23.1, U9.6 (A)
- new net DRV_485B: J4.4 (Pin_4), R23.2, U9.7 (B)
- new net DRV_ALM: R20.2
- new net DRV_ALM_IN: J4.6 (Pin_6), R17.2, R20.1
- new net DRV_DIR+: J5.3 (Pin_3), U10.6 (2Y)
- new net DRV_PU+: J5.1 (Pin_1), U10.3 (1Y)
- new net DRV_RDY: R21.2
- new net DRV_RDY_IN: J4.7 (Pin_7), R18.2, R21.1
- new net DRV_ZO: R22.2
- new net DRV_ZO_IN: J4.8 (Pin_8), R19.2, R22.1
- new net GND: J4.2 (Pin_2), J4.5 (Pin_5), J5.2 (Pin_2), J5.4 (Pin_4), U10.1 (~{1OE}), U10.12 (4A), U10.4 (~{2OE}), U10.7 (GND), U10.9 (3A), U9.5 (GND)
- new net QUAD_A: U10.2 (1A)
- new net QUAD_B: U10.5 (2A)
- new net RS485_DE: U9.2 (~{RE}), U9.3 (DE)
- new net RS485_RX: U9.1 (R)
- new net RS485_TX: U9.4 (D)
Other:
- note added: "DRIVE IO (record sections 11-12; SPEC rulings: 3.3 V RS485 non-isolated, quadrature via 74AHCT125, JST GH signals). Connectors are generic placeholders: operator picks parts and pin order. U9 THVD1450 from a P4 UART in RS485 half-duplex mode; DE and /RE tied, one GPIO. R23 termination fitted-not-populated (short point-to-point run). U10: 3.3 V GPIO in (TTL thresholds), 5 V out to the drive's opto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"
