File: flagship/motor-switch.kicad_sch (KiCad schematic)
At the start: 12 parts, among them J2 BUS_OUT, Q3 B2B_FET_A, Q4 B2B_FET_B, Q5 PRECHARGE_FET, U2 TPS48111LQ1

Commit message: flagship: motor-switch note carries the measured 150 uF drive-side capacitance and the pre-charge numbers
Co-Authored-By: Claude Opus 5.5 (1M context) <noreply@anthropic.com>
Parts:
- removed C5: C_BST, Capacitor_SMD:C_0805_2012Metric, symbol Device:C
- removed C6: C_TMR, Capacitor_SMD:C_0805_2012Metric, symbol Device:C
- removed J2: BUS_OUT, symbol Connector_Generic:Conn_01x02
- removed Q3: B2B_FET_A, symbol Device:Q_NMOS
- removed Q4: B2B_FET_B, symbol Device:Q_NMOS
- removed Q5: PRECHARGE_FET, symbol Device:Q_NMOS
- removed R3: RSNS_MSW, symbol Device:R_Shunt
- removed R4: 100k, Resistor_SMD:R_0805_2012Metric, symbol Device:R
- removed R5, R6: 10k, Resistor_SMD:R_0805_2012Metric, symbol Device:R
- removed R7: R_PRECHARGE, Resistor_SMD:R_2512_6332Metric, symbol Device:R
- removed U2: TPS48111LQ1, flagship:VSSOP-20_19P-L5.0-W3.0-P0.50-LS5.0-BL_PE16, symbol flagship:TPS48111LQDGXRQ1
Other:
- note removed: "MOTOR SWITCH (record section 4). Back-to-back N-FETs, common source, charge pump (TPS4811 integrated 12 V pump: DC on, no bootstrap droop). Open = open both ways: back-drive never reaches the board, which is why the shunt sizes for the powered 6.8 W case. MOTOR_EN floats during P4 boot/reset: R4 pulldown + the chip's internal INP pulldown = off (hard requirement, section 4). INA_ALERT_N on EN/UVL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"

Commit message: flagship: schematic skeleton across all seven sheets
Candidate ICs placed with cross-sheet nets as global labels and a design note per sheet
citing the record: LTC4364IS-2 input protection with INA228 Kelvin shunt and mirrored bulk;
TPS48111 back-to-back motor switch with pre-charge, MOTOR_EN pulldown, INA ALERT hardware
cut; TLV1805 + TLV431 self-acting regen clamp, 2x TO-263, external connector and
parallel/replace jumper; 3x TPS54560B bucks (12/5/3.3 V); Stamp-P4 with fixed pins only
(GPIO assignment follows layout, per ruling); THVD1450 RS485, 74AHCT125 quadrature, drive
status inputs; INA228, thermistor and fan headers. Connectors are generic placeholders.

SPEC.md: rulings for no RP2350 (P4 LP-core emits quadrature) and passive sizes.
Libraries normalized to ASCII (LCSC Chinese manufacturer names, en-dash pin name) after
they broke the MCP server's Windows-codepage reads.

ERC: 109 unconnected pins (detailing), 62 pin-type warnings (LCSC symbols ship
unspecified pin types), 13 one-sided labels (GPIO pending layout); 0 dangling.

Co-Authored-By: Claude Opus 5.5 (1M context) <noreply@anthropic.com>
Parts:
- added C5: C_BST, Capacitor_SMD:C_0805_2012Metric, symbol Device:C
- added C6: C_TMR, Capacitor_SMD:C_0805_2012Metric, symbol Device:C
- added J2: BUS_OUT, symbol Connector_Generic:Conn_01x02
- added Q3: B2B_FET_A, symbol Device:Q_NMOS
- added Q4: B2B_FET_B, symbol Device:Q_NMOS
- added Q5: PRECHARGE_FET, symbol Device:Q_NMOS
- added R3: RSNS_MSW, symbol Device:R_Shunt
- added R4: 100k, Resistor_SMD:R_0805_2012Metric, symbol Device:R
- added R5, R6: 10k, Resistor_SMD:R_0805_2012Metric, symbol Device:R
- added R7: R_PRECHARGE, Resistor_SMD:R_2512_6332Metric, symbol Device:R
- added U2: TPS48111LQ1, flagship:VSSOP-20_19P-L5.0-W3.0-P0.50-LS5.0-BL_PE16, symbol flagship:TPS48111LQDGXRQ1
Connections:
- new net +3V3: R5.1, R6.1
- new net +BUS: R3.1, U2.20 (VS)
- new net GND: C6.2, J2.2 (Pin_2), R4.2, U2.6 (GND)
- new net INA_ALERT_N: R5.2, U2.1 (EN/UVLO)
- new net MOTOR_EN: R4.1, U2.3 (INP)
- new net MOTOR_V+: J2.1 (Pin_1)
- new net MSW_BST: C5.1, U2.12 (BST)
- new net MSW_CS+: R3.2, U2.18 (CS+)
- new net MSW_CS-: R3.3, U2.17 (CS-)
- new net MSW_FLT_N: R6.2, U2.4 (~{FLT_T}), U2.5 (~{FLT_I})
- new net MSW_IMON: U2.7 (IMON)
- new net MSW_SRC: C5.2, U2.13 (SRC)
- new net MSW_TMR: C6.1, U2.9 (TMR)
- new net PRECHARGE_EN: U2.2 (INP_G)
Other:
- note added: "MOTOR SWITCH (record section 4). Back-to-back N-FETs, common source, charge pump (TPS4811 integrated 12 V pump: DC on, no bootstrap droop). Open = open both ways: back-drive never reaches the board, which is why the shunt sizes for the powered 6.8 W case. MOTOR_EN floats during P4 boot/reset: R4 pulldown + the chip's internal INP pulldown = off (hard requirement, section 4). INA_ALERT_N on EN/UVL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"
