File: flagship/motor-switch.kicad_sch (KiCad schematic)
At the start: 12 parts, among them J2 BUS_OUT, Q3 B2B_FET_A, Q4 B2B_FET_B, Q5 PRECHARGE_FET, U2 TPS48111LQ1

Commit message: flagship: rails detailed per the TPS54560B datasheet; logic power moved to the stamp's own rails
Rails: three identical 400 kHz columns (A3 sheet), 4 A each, VIN 20-48 V, UVLO 20/17 V,
values from the datasheet design procedure (inductor, derated ceramic output, FB, type-II
comp, B560C catch diode, 4x 2.2u/100V input). Worst on-time 205 ns vs 135 ns minimum.
Logic power (operator): +5V_SYS = stamp pad 39 (VIN/USB OR) feeds the 74AHCT125, drive
485_5V and status LED, so USB alone emits quadrature; +3V3_SYS = stamp pad 28 feeds the
INA228, THVD1450 and all pull-ups. 3.3 V buck is accessory-only (+3V3_ACC). Netlist checked:
the five power domains are separate. SPEC rulings recorded.

Co-Authored-By: Claude Opus 5.5 (1M context) <noreply@anthropic.com>
Connections:
- net +3V3 renamed +3V3_SYS
Changed lines of the file:
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@@
 		)
 	)
-	(global_label "+3V3"
+	(global_label "+3V3_SYS"
 		(shape bidirectional)
 		(at 69.85 135.89 90)
@@
 		)
 	)
-	(global_label "+3V3"
+	(global_label "+3V3_SYS"
 		(shape bidirectional)
 		(at 54.61 135.89 90)
