File: flagship/rails.kicad_sch (KiCad schematic)
At the start: 15 parts, among them U5 TPS54560B, U6 TPS54560B, U7 TPS54560B

Commit message: flagship: motor-switch note carries the measured 150 uF drive-side capacitance and the pre-charge numbers
Co-Authored-By: Claude Opus 5.5 (1M context) <noreply@anthropic.com>
Parts:
- removed C10: COUT_5V, Capacitor_SMD:C_1210_3225Metric, symbol Device:C
- removed C11, C7, C9: BOOT_0.1u, Capacitor_SMD:C_0805_2012Metric, symbol Device:C
- removed C12: COUT_3V3, Capacitor_SMD:C_1210_3225Metric, symbol Device:C
- removed C8: COUT_12V, Capacitor_SMD:C_1210_3225Metric, symbol Device:C
- removed D2, D3, D4: SS560, symbol Device:D_Schottky
- removed L1: L_12V, symbol Device:L
- removed L2: L_5V, symbol Device:L
- removed L3: L_3V3, symbol Device:L
- removed U5, U6, U7: TPS54560B, flagship:POWERPAD-SO-8_L4.9-W3.9-P1.27-LS6.0-BL-EP, symbol flagship:TPS54560BDDAR
Other:
- note removed: "RAILS (record section 10): independent bucks from +BUS, the record's "likely" topology. TPS54560B x3: 60 V in, 5 A, SO-8 PowerPAD (gull-wing, hand-solderable), one design laid out three times. Input headroom: bus clamps at ~45 V, part is rated 60 V. +12V: regen clamp supply (must self-start, no enable from firmware), fan, accessory 12 V. +5V: stamp VIN (pin 14; stamp makes its own 3.3 V for the P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"

Commit message: flagship: schematic skeleton across all seven sheets
Candidate ICs placed with cross-sheet nets as global labels and a design note per sheet
citing the record: LTC4364IS-2 input protection with INA228 Kelvin shunt and mirrored bulk;
TPS48111 back-to-back motor switch with pre-charge, MOTOR_EN pulldown, INA ALERT hardware
cut; TLV1805 + TLV431 self-acting regen clamp, 2x TO-263, external connector and
parallel/replace jumper; 3x TPS54560B bucks (12/5/3.3 V); Stamp-P4 with fixed pins only
(GPIO assignment follows layout, per ruling); THVD1450 RS485, 74AHCT125 quadrature, drive
status inputs; INA228, thermistor and fan headers. Connectors are generic placeholders.

SPEC.md: rulings for no RP2350 (P4 LP-core emits quadrature) and passive sizes.
Libraries normalized to ASCII (LCSC Chinese manufacturer names, en-dash pin name) after
they broke the MCP server's Windows-codepage reads.

ERC: 109 unconnected pins (detailing), 62 pin-type warnings (LCSC symbols ship
unspecified pin types), 13 one-sided labels (GPIO pending layout); 0 dangling.

Co-Authored-By: Claude Opus 5.5 (1M context) <noreply@anthropic.com>
Parts:
- added C10: COUT_5V, Capacitor_SMD:C_1210_3225Metric, symbol Device:C
- added C11, C7, C9: BOOT_0.1u, Capacitor_SMD:C_0805_2012Metric, symbol Device:C
- added C12: COUT_3V3, Capacitor_SMD:C_1210_3225Metric, symbol Device:C
- added C8: COUT_12V, Capacitor_SMD:C_1210_3225Metric, symbol Device:C
- added D2, D3, D4: SS560, symbol Device:D_Schottky
- added L1: L_12V, symbol Device:L
- added L2: L_5V, symbol Device:L
- added L3: L_3V3, symbol Device:L
- added U5, U6, U7: TPS54560B, flagship:POWERPAD-SO-8_L4.9-W3.9-P1.27-LS6.0-BL-EP, symbol flagship:TPS54560BDDAR
Connections:
- new net +12V: C8.1, L1.2
- new net +3V3: C12.1, L3.2
- new net +5V: C10.1, L2.2
- new net +BUS: U5.2 (VIN), U6.2 (VIN), U7.2 (VIN)
- new net BOOT_12V: C7.1, U5.1 (BOOT)
- new net BOOT_3V3: C11.1, U7.1 (BOOT)
- new net BOOT_5V: C9.1, U6.1 (BOOT)
- new net GND: C10.2, C12.2, C8.2, D2.2 (A), D3.2 (A), D4.2 (A), U5.7 (GND), U5.9 (EP), U6.7 (GND), U6.9 (EP), U7.7 (GND), U7.9 (EP)
- new net SW_12V: C7.2, D2.1 (K), L1.1, U5.8 (SW)
- new net SW_3V3: C11.2, D4.1 (K), L3.1, U7.8 (SW)
- new net SW_5V: C9.2, D3.1 (K), L2.1, U6.8 (SW)
Other:
- note added: "RAILS (record section 10): independent bucks from +BUS, the record's "likely" topology. TPS54560B x3: 60 V in, 5 A, SO-8 PowerPAD (gull-wing, hand-solderable), one design laid out three times. Input headroom: bus clamps at ~45 V, part is rated 60 V. +12V: regen clamp supply (must self-start, no enable from firmware), fan, accessory 12 V. +5V: stamp VIN (pin 14; stamp makes its own 3.3 V for the P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"
