File: flagship/rails.kicad_sch (KiCad schematic)
At the start: 15 parts, among them U5 TPS54560B, U6 TPS54560B, U7 TPS54560B

Commit message: flagship: rails detailed per the TPS54560B datasheet; logic power moved to the stamp's own rails
Rails: three identical 400 kHz columns (A3 sheet), 4 A each, VIN 20-48 V, UVLO 20/17 V,
values from the datasheet design procedure (inductor, derated ceramic output, FB, type-II
comp, B560C catch diode, 4x 2.2u/100V input). Worst on-time 205 ns vs 135 ns minimum.
Logic power (operator): +5V_SYS = stamp pad 39 (VIN/USB OR) feeds the 74AHCT125, drive
485_5V and status LED, so USB alone emits quadrature; +3V3_SYS = stamp pad 28 feeds the
INA228, THVD1450 and all pull-ups. 3.3 V buck is accessory-only (+3V3_ACC). Netlist checked:
the five power domains are separate. SPEC rulings recorded.

Co-Authored-By: Claude Opus 5.5 (1M context) <noreply@anthropic.com>
Parts:
- removed C10: COUT_5V, Capacitor_SMD:C_1210_3225Metric, symbol Device:C
- removed C11, C7, C9: BOOT_0.1u, Capacitor_SMD:C_0805_2012Metric, symbol Device:C
- removed C12: COUT_3V3, Capacitor_SMD:C_1210_3225Metric, symbol Device:C
- removed C8: COUT_12V, Capacitor_SMD:C_1210_3225Metric, symbol Device:C
- added C101, C102, C103, C104, C201, C202, C203, C204, C301, C302, C303, C304: 2.2u 100V, Capacitor_SMD:C_1210_3225Metric, symbol Device:C
- added C105: 5.6n, Capacitor_SMD:C_0805_2012Metric, symbol Device:C
- added C106, C206, C306: DNP, Capacitor_SMD:C_0805_2012Metric, symbol Device:C
- added C107, C207, C307: 0.1u, Capacitor_SMD:C_0805_2012Metric, symbol Device:C
- added C108, C109, C110, C111: 22u 25V, Capacitor_SMD:C_1210_3225Metric, symbol Device:C
- added C205, C305: 6.8n, Capacitor_SMD:C_0805_2012Metric, symbol Device:C
- added C208, C209, C210, C308, C309, C310: 47u 10V, Capacitor_SMD:C_1210_3225Metric, symbol Device:C
- added R101, R201, R301: 887k, Resistor_SMD:R_0805_2012Metric, symbol Device:R
- added R102, R202, R302: 53.6k, Resistor_SMD:R_0805_2012Metric, symbol Device:R
- added R103, R203, R303: 243k, Resistor_SMD:R_0805_2012Metric, symbol Device:R
- added R104: 21.5k, Resistor_SMD:R_0805_2012Metric, symbol Device:R
- added R105: 140k, Resistor_SMD:R_0805_2012Metric, symbol Device:R
- added R106, R206, R306: 10k, Resistor_SMD:R_0805_2012Metric, symbol Device:R
- added R204: 15.8k, Resistor_SMD:R_0805_2012Metric, symbol Device:R
- added R205: 52.3k, Resistor_SMD:R_0805_2012Metric, symbol Device:R
- added R304: 13.7k, Resistor_SMD:R_0805_2012Metric, symbol Device:R
- added R305: 31.6k, Resistor_SMD:R_0805_2012Metric, symbol Device:R
- D2, D3, D4: value SS560 -> B560C; footprint (none) -> Diode_SMD:D_SMC
- L1: value L_12V -> 18u Isat>=7.5A
- L2: value L_5V -> 10u Isat>=7.5A
- L3: value L_3V3 -> 6.8u Isat>=7.5A
- U5: value TPS54560B -> TPS54560B 12V
- U6: value TPS54560B -> TPS54560B 5V
- U7: value TPS54560B -> TPS54560B 3V3
Connections:
- net +12V: now also C108.1, C109.1, C110.1, C111.1, R105.1
- net +5V: now also C208.1, C209.1, C210.1, R205.1
- net +BUS: now also C101.1, C102.1, C103.1, C104.1, C201.1, C202.1, C203.1, C204.1, C301.1, C302.1, C303.1, C304.1, R101.1, R201.1, R301.1
- net BOOT_12V: now also C107.1
- net BOOT_3V3: now also C307.1
- net BOOT_5V: now also C207.1
- net GND: now also C101.2, C102.2, C103.2, C104.2, C105.2, C106.2, C108.2, C109.2, C110.2, C111.2, C201.2, C202.2, C203.2, C204.2, C205.2, C206.2, C208.2, C209.2, C210.2, C301.2, C302.2, C303.2, C304.2, C305.2, C306.2, C308.2, C309.2, C310.2, R102.2, R103.2, R106.2, R202.2, R203.2, R206.2, R302.2, R303.2, R306.2
- net SW_12V: now also C107.2
- net SW_3V3: now also C307.2
- net SW_5V: now also C207.2
- net EN_12V: now reaches U5.3 (EN)
- net EN_12V: now also R101.2, R102.1
- net RT_12V: now reaches U5.4 (RT/CLK)
- net RT_12V: now also R103.1
- net FB_12V: now reaches U5.5 (FB)
- net FB_12V: now also R105.2, R106.1
- net COMP_12V: now reaches U5.6 (COMP)
- net COMP_12V: now also C106.1, R104.1
- net EN_3V3: now reaches U7.3 (EN)
- net EN_3V3: now also R301.2, R302.1
- net RT_3V3: now reaches U7.4 (RT/CLK)
- net RT_3V3: now also R303.1
- net FB_3V3: now reaches U7.5 (FB)
- net FB_3V3: now also R305.2, R306.1
- net COMP_3V3: now reaches U7.6 (COMP)
- net COMP_3V3: now also C306.1, R304.1
- net EN_5V: now reaches U6.3 (EN)
- net EN_5V: now also R201.2, R202.1
- net RT_5V: now reaches U6.4 (RT/CLK)
- net RT_5V: now also R203.1
- net FB_5V: now reaches U6.5 (FB)
- net FB_5V: now also R205.2, R206.1
- net COMP_5V: now reaches U6.6 (COMP)
- net COMP_5V: now also C206.1, R204.1
- net +3V3 renamed +3V3_ACC
- net +3V3_ACC: now also C308.1, C309.1, C310.1, R305.1
- new net COMPZ_12V: C105.1, R104.2
- new net COMPZ_3V3: C305.1, R304.2
- new net COMPZ_5V: C205.1, R204.2
Other:
- note added: "RAILS (record section 10: independent bucks from +BUS). TPS54560B x3, one layout three times; values from the datasheet's own design procedure (SLVSF00 section 8.2). Design inputs: VIN 20-48 V (48 = supply OVP ceiling, covers the ~45 V clamp; part rated 60 V), 4 A per rail, 400 kHz, half-load step held within 4 %. fsw 400 kHz: RT 243k. Worst on-time 3.3 V at 48 V = 205 ns vs 135 ns minimum. UVLO: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"
- note removed: "RAILS (record section 10): independent bucks from +BUS, the record's "likely" topology. TPS54560B x3: 60 V in, 5 A, SO-8 PowerPAD (gull-wing, hand-solderable), one design laid out three times. Input headroom: bus clamps at ~45 V, part is rated 60 V. +12V: regen clamp supply (must self-start, no enable from firmware), fan, accessory 12 V. +5V: stamp VIN (pin 14; stamp makes its own 3.3 V for the P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"

Commit message: flagship: drop the duplicate GND power flag on the rails sheet (ERC power-output clash)
Co-Authored-By: Claude Opus 5.5 (1M context) <noreply@anthropic.com>
Changed lines of the file:
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@@
-	(global_label "GND"
-		(shape bidirectional)
-		(at 415.29 49.53 270)
-		(effects
-			(font
-				(size 1.27 1.27)
-			)
-			(justify right)
-		)
-		(property "Intersheetrefs" "${INTERSHEET_REFS}"
-			(at 415.29 49.53 0)
-			(hide yes)
-			(show_name no)
-			(do_not_autoplace no)
-			(effects
-				(font
-					(size 1.27 1.27)
-				)
-			)
-		)
-	)
 	(global_label "GND"
 		(shape bidirectional)
@@
 					(unit 1)
 				)
-			)
-		)
-	)
-	(symbol
-		(lib_id "power:PWR_FLAG")
-		(at 415.29 49.53 0)
-		(unit 1)
-		(body_style 1)
-		(exclude_from_sim no)
-		(in_bom yes)
-		(on_board yes)
-		(in_pos_files yes)
-		(dnp no)
-		(property "Reference" "#FLG302"
-			(at 415.29 46.99 0)
-			(show_name no)
-			(do_not_autoplace no)
-			(effects
-				(font
-					(size 1.27 1.27)
-				)
-			)
-		)
-		(property "Value" "PWR_FLAG"
-			(at 415.29 52.07 0)
-			(show_name no)
-			(do_not_autoplace no)
-			(effects
-				(font
-					(size 1.27 1.27)
-				)
-			)
-		)
-		(property "Footprint" ""
-			(at 415.29 49.53 0)
-			(hide yes)
-			(show_name no)
-			(do_not_autoplace no)
-			(effects
-				(font
-					(size 1.27 1.27)
-				)
-			)
-		)
-		(property "Datasheet" ""
-			(at 415.29 49.53 0)
-			(hide yes)
-			(show_name no)
-			(do_not_autoplace no)
-			(effects
-				(font
-					(size 1.27 1.27)
-				)
-			)
-		)
-		(property "Description" "Special symbol for telling ERC where power comes from"
-			(at 415.29 49.53 0)
-			(hide yes)
-			(show_name no)
-			(do_not_autoplace no)
-			(effects
-				(font
-					(size 1.27 1.27)
-				)
-			)
-		)
-		(pin "1"
-		)
-		(instances
-			(project ""
-				(path "/f57caae8-afe4-4c0e-ae57-d0e1c6b942e6"
-					(reference "#FLG302")
-					(unit 1)
-				)
