File: flagship/regen-shunt.kicad_sch (KiCad schematic)
At the start: 15 parts, among them J3 EXT_SHUNT, Q6 CLAMP_FET_100V, U3 TLV1805, U4 TLV431

Commit message: flagship: motor-switch note carries the measured 150 uF drive-side capacitance and the pre-charge numbers
Co-Authored-By: Claude Opus 5.5 (1M context) <noreply@anthropic.com>
Parts:
- removed D1: TVS_SHUNT, symbol Device:D_TVS
- removed J3: EXT_SHUNT, symbol Connector_Generic:Conn_01x02
- removed JP1: CUT=EXT_ONLY, symbol Jumper:SolderJumper_2_Bridged
- removed Q6: CLAMP_FET_100V, symbol Device:Q_NMOS
- removed R10: R_HYST, Resistor_SMD:R_0805_2012Metric, symbol Device:R
- removed R11, R12: 16R_TO263, symbol Device:R
- removed R13: 10k, Resistor_SMD:R_0805_2012Metric, symbol Device:R
- removed R14: 3.3k, Resistor_SMD:R_0805_2012Metric, symbol Device:R
- removed R15: 10R, Resistor_SMD:R_0805_2012Metric, symbol Device:R
- removed R16: R_REF_BIAS, Resistor_SMD:R_0805_2012Metric, symbol Device:R
- removed R8: R_DIV_TOP, Resistor_SMD:R_1206_3216Metric, symbol Device:R
- removed R9: R_DIV_BOT, Resistor_SMD:R_0805_2012Metric, symbol Device:R
- removed U3: TLV1805, flagship:TSOT-23-6_L2.9-W1.6-P0.95-LS2.8-BL, symbol flagship:TLV1805DBVR
- removed U4: TLV431, flagship:SOT-23-3_L2.9-W1.3-P1.90-LS2.4-BR, symbol flagship:TLV431AIDBZR
Other:
- note removed: "REGEN SHUNT (record section 5). Self-acting clamp: comparator + reference + FET, no firmware in the loop. Threshold ~45 V ON, a few volts hysteresis. That is above the GST360A36 worst-case 37.8 V OVP trip, legal ONLY because the input section blocks reverse current: the supply never sees the bus rise. Sizing ~7 W continuous / ~150 W peak (motor switch removes the unpowered case). R11 || R12: two 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"

Commit message: flagship: schematic skeleton across all seven sheets
Candidate ICs placed with cross-sheet nets as global labels and a design note per sheet
citing the record: LTC4364IS-2 input protection with INA228 Kelvin shunt and mirrored bulk;
TPS48111 back-to-back motor switch with pre-charge, MOTOR_EN pulldown, INA ALERT hardware
cut; TLV1805 + TLV431 self-acting regen clamp, 2x TO-263, external connector and
parallel/replace jumper; 3x TPS54560B bucks (12/5/3.3 V); Stamp-P4 with fixed pins only
(GPIO assignment follows layout, per ruling); THVD1450 RS485, 74AHCT125 quadrature, drive
status inputs; INA228, thermistor and fan headers. Connectors are generic placeholders.

SPEC.md: rulings for no RP2350 (P4 LP-core emits quadrature) and passive sizes.
Libraries normalized to ASCII (LCSC Chinese manufacturer names, en-dash pin name) after
they broke the MCP server's Windows-codepage reads.

ERC: 109 unconnected pins (detailing), 62 pin-type warnings (LCSC symbols ship
unspecified pin types), 13 one-sided labels (GPIO pending layout); 0 dangling.

Co-Authored-By: Claude Opus 5.5 (1M context) <noreply@anthropic.com>
Parts:
- added D1: TVS_SHUNT, symbol Device:D_TVS
- added J3: EXT_SHUNT, symbol Connector_Generic:Conn_01x02
- added JP1: CUT=EXT_ONLY, symbol Jumper:SolderJumper_2_Bridged
- added Q6: CLAMP_FET_100V, symbol Device:Q_NMOS
- added R10: R_HYST, Resistor_SMD:R_0805_2012Metric, symbol Device:R
- added R11, R12: 16R_TO263, symbol Device:R
- added R13: 10k, Resistor_SMD:R_0805_2012Metric, symbol Device:R
- added R14: 3.3k, Resistor_SMD:R_0805_2012Metric, symbol Device:R
- added R15: 10R, Resistor_SMD:R_0805_2012Metric, symbol Device:R
- added R16: R_REF_BIAS, Resistor_SMD:R_0805_2012Metric, symbol Device:R
- added R8: R_DIV_TOP, Resistor_SMD:R_1206_3216Metric, symbol Device:R
- added R9: R_DIV_BOT, Resistor_SMD:R_0805_2012Metric, symbol Device:R
- added U3: TLV1805, flagship:TSOT-23-6_L2.9-W1.6-P0.95-LS2.8-BL, symbol flagship:TLV1805DBVR
- added U4: TLV431, flagship:SOT-23-3_L2.9-W1.3-P1.90-LS2.4-BR, symbol flagship:TLV431AIDBZR
Connections:
- new net +12V: R16.1, U3.6 (V+)
- new net +BUS: J3.1 (Pin_1), R11.1, R12.1, R8.1
- new net BUS_DIV: R10.1, R8.2, R9.1, U3.4 (+IN)
- new net CLAMP_G: Q6.G, R15.2
- new net CLAMP_GATE: R10.2, R13.1, R15.1, U3.1 (OUT)
- new net CLAMP_MON: R13.2, R14.1
- new net GND: D1.2 (A2), Q6.S, R14.2, R9.2, U3.2 (V-), U4.3 (A)
- new net SHUNT_ARRAY: JP1.1 (A), R11.2, R12.2
- new net SHUNT_SW: D1.1 (A1), J3.2 (Pin_2), JP1.2 (B), Q6.D
- new net VREF: R16.2, U3.3 (-IN), U4.1 (REF), U4.2 (C)
Other:
- note added: "REGEN SHUNT (record section 5). Self-acting clamp: comparator + reference + FET, no firmware in the loop. Threshold ~45 V ON, a few volts hysteresis. That is above the GST360A36 worst-case 37.8 V OVP trip, legal ONLY because the input section blocks reverse current: the supply never sees the bus rise. Sizing ~7 W continuous / ~150 W peak (motor switch removes the unpowered case). R11 || R12: two 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"
