File: flagship/sensing.kicad_sch (KiCad schematic)
At the start: 12 parts, among them J6 THERMISTOR, J7 FAN_4PIN, U11 INA228

Commit message: flagship: motor-switch note carries the measured 150 uF drive-side capacitance and the pre-charge numbers
Co-Authored-By: Claude Opus 5.5 (1M context) <noreply@anthropic.com>
Parts:
- removed C13, C14: 0.1u, Capacitor_SMD:C_0805_2012Metric, symbol Device:C
- removed J6: THERMISTOR, symbol Connector_Generic:Conn_01x02
- removed J7: FAN_4PIN, symbol Connector_Generic:Conn_01x04
- removed JP2: FAN_V_12V|5V, symbol Jumper:SolderJumper_3_Open
- removed R24, R25: 4.7k, Resistor_SMD:R_0805_2012Metric, symbol Device:R
- removed R26, R28: 10k, Resistor_SMD:R_0805_2012Metric, symbol Device:R
- removed R27, R29: 1k, Resistor_SMD:R_0805_2012Metric, symbol Device:R
- removed U11: INA228, flagship:VSSOP-10_L3.0-W3.0-P0.50-LS4.9-BL, symbol flagship:INA228AIDGSR
Other:
- note removed: "SENSING (record sections 10, 12). U11 INA228 across R2 on the Input sheet via Kelvin taps INA_SENSE_P/N: route as a tight pair, INA beside the shunt, quiet ground, far from switch nodes. 1 mOhm: 10 mV at 10 A, inside the +-163.84 mV range; die temperature = board temperature (the thermal witness per the heatsink ruling). ALERT (open drain) = INA_ALERT_N: also the motor switch EN/UVLO, so over-cur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"
