File: flagship/compute.kicad_sch (KiCad schematic)
At the start: 0 parts

Commit message: flagship: schematic skeleton across all seven sheets
Candidate ICs placed with cross-sheet nets as global labels and a design note per sheet
citing the record: LTC4364IS-2 input protection with INA228 Kelvin shunt and mirrored bulk;
TPS48111 back-to-back motor switch with pre-charge, MOTOR_EN pulldown, INA ALERT hardware
cut; TLV1805 + TLV431 self-acting regen clamp, 2x TO-263, external connector and
parallel/replace jumper; 3x TPS54560B bucks (12/5/3.3 V); Stamp-P4 with fixed pins only
(GPIO assignment follows layout, per ruling); THVD1450 RS485, 74AHCT125 quadrature, drive
status inputs; INA228, thermistor and fan headers. Connectors are generic placeholders.

SPEC.md: rulings for no RP2350 (P4 LP-core emits quadrature) and passive sizes.
Libraries normalized to ASCII (LCSC Chinese manufacturer names, en-dash pin name) after
they broke the MCP server's Windows-codepage reads.

ERC: 109 unconnected pins (detailing), 62 pin-type warnings (LCSC symbols ship
unspecified pin types), 13 one-sided labels (GPIO pending layout); 0 dangling.

Co-Authored-By: Claude Opus 5.5 (1M context) <noreply@anthropic.com>
Parts:
- added D5: STATUS_RGB, LED_SMD:LED_WS2812B_PLCC4_5.0x5.0mm_P3.2mm, symbol LED:WS2812B
- added SW1: RESET, symbol Switch:SW_Push
- added SW2: BOOT, symbol Switch:SW_Push
- added U8: Stamp-P4, flagship:Stamp-P4, symbol m5stack:Stamp-P4
Connections:
- new net +5V: D5.1 (VDD), U8.14 (VIN)
- new net GND: D5.3 (VSS), SW1.2, SW2.2, U8.13 (GND), U8.38 (GND), U8.42 (GND), U8.56 (GND), U8.59 (GND), U8.62 (GND), U8.65 (GND)
- new net LED_DATA: D5.4 (DIN)
- new net P4_BOOT: SW2.1, U8.36 (G35_BOOT_RMII_TXD1), U8.48 (G35_BOOT_RMII_TXD1)
- new net P4_EN: SW1.1, U8.34 (CHIP_EN)
Other:
- note added: "COMPUTE (record section 8; SPEC: no RP2350, the P4 LP core emits quadrature). Stamp-P4 + Stamp-AddOn C6 stacked on top (SDIO G42-G48, not castellated). Fixed pins only: VIN (14) from +5V, the stamp ORs it with its own USB-C 5V and makes SOC_3.3V itself; all GND pads; CHIP_EN + G35 buttons (stamp has 10k pull-ups). G35 appears on pads 36 AND 48 in M5's own symbol and schematic: both wired to P4_BO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"

Commit message: flagship: rails detailed per the TPS54560B datasheet; logic power moved to the stamp's own rails
Rails: three identical 400 kHz columns (A3 sheet), 4 A each, VIN 20-48 V, UVLO 20/17 V,
values from the datasheet design procedure (inductor, derated ceramic output, FB, type-II
comp, B560C catch diode, 4x 2.2u/100V input). Worst on-time 205 ns vs 135 ns minimum.
Logic power (operator): +5V_SYS = stamp pad 39 (VIN/USB OR) feeds the 74AHCT125, drive
485_5V and status LED, so USB alone emits quadrature; +3V3_SYS = stamp pad 28 feeds the
INA228, THVD1450 and all pull-ups. 3.3 V buck is accessory-only (+3V3_ACC). Netlist checked:
the five power domains are separate. SPEC rulings recorded.

Co-Authored-By: Claude Opus 5.5 (1M context) <noreply@anthropic.com>
Connections:
- net +5V: no longer D5.1 (VDD)
- net +3V3_SYS: now reaches U8.28 (SOC_3.3V)
- net +5V_SYS: now reaches U8.39 (SYS_5V)
- net +5V_SYS: now also D5.1 (VDD)
Changed lines of the file:
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@@
+		)
+	)
+	(global_label "+5V_SYS"
+		(shape bidirectional)
+		(at 240.03 142.24 90)
+		(effects
+			(font
+				(size 1.27 1.27)
+			)
+			(justify left)
+		)
+		(property "Intersheetrefs" "${INTERSHEET_REFS}"
+			(at 240.03 142.24 0)
+			(hide yes)
+			(show_name no)
+			(do_not_autoplace no)
+			(effects
+				(font
+					(size 1.27 1.27)
+				)
+			)
 		)
 	)
@@
 		)
 	)
+	(global_label "+3V3_SYS"
+		(shape bidirectional)
+		(at 74.93 100.33 270)
+		(effects
+			(font
+				(size 1.27 1.27)
+			)
+			(justify right)
+		)
+		(property "Intersheetrefs" "${INTERSHEET_REFS}"
+			(at 74.93 100.33 0)
+			(hide yes)
+			(show_name no)
+			(do_not_autoplace no)
+			(effects
+				(font
+					(size 1.27 1.27)
+				)
+			)
+		)
+	)
 	(global_label "GND"
 		(shape bidirectional)
@@
 		)
 	)
+	(global_label "+3V3_SYS"
+		(shape bidirectional)
+		(at 102.87 85.09 180)
+		(effects
+			(font
+				(size 1.27 1.27)
+			)
+			(justify right)
+		)
+		(property "Intersheetrefs" "${INTERSHEET_REFS}"
+			(at 102.87 85.09 0)
+			(hide yes)
+			(show_name no)
+			(do_not_autoplace no)
+			(effects
+				(font
+					(size 1.27 1.27)
+				)
+			)
+		)
+	)
+	(global_label "+5V_SYS"
+		(shape bidirectional)
+		(at 59.69 100.33 270)
+		(effects
+			(font
+				(size 1.27 1.27)
+			)
+			(justify right)
+		)
+		(property "Intersheetrefs" "${INTERSHEET_REFS}"
+			(at 59.69 100.33 0)
+			(hide yes)
+			(show_name no)
+			(do_not_autoplace no)
+			(effects
+				(font
+					(size 1.27 1.27)
+				)
+			)
+		)
+	)
+	(global_label "+5V_SYS"
+		(shape bidirectional)
+		(at 102.87 87.63 180)
+		(effects
+			(font
+				(size 1.27 1.27)
+			)
+			(justify right)
+		)
+		(property "Intersheetrefs" "${INTERSHEET_REFS}"
+			(at 102.87 87.63 0)
+			(hide yes)
+			(show_name no)
+			(do_not_autoplace no)
+			(effects
+				(font
+					(size 1.27 1.27)
+				)
+			)
+		)
+	)
 	(global_label "+5V"
 		(shape bidirectional)
@@
 		(property "Intersheetrefs" "${INTERSHEET_REFS}"
 			(at 102.87 97.79 0)
-			(hide yes)
-			(show_name no)
-			(do_not_autoplace no)
-			(effects
-				(font
-					(size 1.27 1.27)
-				)
-			)
-		)
-	)
-	(global_label "+5V"
-		(shape bidirectional)
-		(at 240.03 142.24 90)
-		(effects
-			(font
-				(size 1.27 1.27)
-			)
-			(justify left)
-		)
-		(property "Intersheetrefs" "${INTERSHEET_REFS}"
-			(at 240.03 142.24 0)
 			(hide yes)
 			(show_name no)
@@
 					(unit 1)
 				)
+			)
+		)
+	)
+	(symbol
+		(lib_id "power:PWR_FLAG")
+		(at 74.93 100.33 0)
+		(unit 1)
+		(body_style 1)
+		(exclude_from_sim no)
+		(in_bom yes)
+		(on_board yes)
+		(in_pos_files yes)
+		(dnp no)
+		(property "Reference" "#FLG402"
+			(at 74.93 97.79 0)
+			(show_name no)
+			(do_not_autoplace no)
+			(effects
+				(font
+					(size 1.27 1.27)
+				)
+			)
+		)
+		(property "Value" "PWR_FLAG"
+			(at 74.93 102.87 0)
+			(show_name no)
+			(do_not_autoplace no)
+			(effects
+				(font
+					(size 1.27 1.27)
+				)
+			)
+		)
+		(property "Footprint" ""
+			(at 74.93 100.33 0)
+			(hide yes)
+			(show_name no)
+			(do_not_autoplace no)
+			(effects
+				(font
+					(size 1.27 1.27)
+				)
+			)
+		)
+		(property "Datasheet" ""
+			(at 74.93 100.33 0)
+			(hide yes)
+			(show_name no)
+			(do_not_autoplace no)
+			(effects
+				(font
+					(size 1.27 1.27)
+				)
+			)
+		)
+		(property "Description" "Special symbol for telling ERC where power comes from"
+			(at 74.93 100.33 0)
+			(hide yes)
+			(show_name no)
+			(do_not_autoplace no)
+			(effects
+				(font
+					(size 1.27 1.27)
+				)
+			)
+		)
+		(pin "1"
+		)
+		(instances
+			(project ""
+				(path "/c8d93a19-1a8c-428f-b3f5-f89cc40da3c2"
+					(reference "#FLG402")
+					(unit 1)
+				)
+			)
+		)
+	)
+	(symbol
+		(lib_id "power:PWR_FLAG")
+		(at 59.69 100.33 0)
+		(unit 1)
+		(body_style 1)
+		(exclude_from_sim no)
+		(in_bom yes)
+		(on_board yes)
+		(in_pos_files yes)
+		(dnp no)
+		(property "Reference" "#FLG401"
+			(at 59.69 97.79 0)
+			(show_name no)
+			(do_not_autoplace no)
+			(effects
+				(font
+					(size 1.27 1.27)
+				)
+			)
+		)
+		(property "Value" "PWR_FLAG"
+			(at 59.69 102.87 0)
+			(show_name no)
+			(do_not_autoplace no)
+			(effects
+				(font
+					(size 1.27 1.27)
+				)
+			)
+		)
+		(property "Footprint" ""
+			(at 59.69 100.33 0)
+			(hide yes)
+			(show_name no)
+			(do_not_autoplace no)
+			(effects
+				(font
+					(size 1.27 1.27)
+				)
+			)
+		)
+		(property "Datasheet" ""
+			(at 59.69 100.33 0)
+			(hide yes)
+			(show_name no)
+			(do_not_autoplace no)
+			(effects
+				(font
+					(size 1.27 1.27)
+				)
+			)
+		)
+		(property "Description" "Special symbol for telling ERC where power comes from"
+			(at 59.69 100.33 0)
+			(hide yes)
+			(show_name no)
+			(do_not_autoplace no)
+			(effects
+				(font
+					(size 1.27 1.27)
+				)
+			)
+		)
+		(pin "1"
+		)
+		(instances
+			(project ""
+				(path "/c8d93a19-1a8c-428f-b3f5-f89cc40da3c2"
+					(reference "#FLG401")
+					(unit 1)
+				)
