File: flagship/compute.kicad_sch (KiCad schematic)
At the start: 4 parts, among them SW1 RESET, SW2 BOOT, U8 Stamp-P4

Commit message: flagship: drive connectors (XT30 + GH4 motion / XT30 ext shunt + GH6 comms), HOME and PAIR buttons with EN/BOOT rescue pads, status LED through AHCT125 gate 3, ZO dropped; FEATURES.md
ZO removal: DRV_ZO / DRV_ZO_IN and R19/R22 existed only on the Drive IO sheet (netlist checked: no other node on either net).
Parts:
- added TP901: EN, TestPoint:TestPoint_Pad_D1.5mm, symbol Connector:TestPoint
- added TP902: GND, TestPoint:TestPoint_Pad_D1.5mm, symbol Connector:TestPoint
- added TP903: BOOT, TestPoint:TestPoint_Pad_D1.5mm, symbol Connector:TestPoint
- SW1: value RESET -> HOME (hold: RESET)
- SW2: value BOOT -> PAIR (held at power-on: AP)
Connections:
- net GND: now also TP902.1
- net P4_BOOT: now also TP903.1; no longer SW2.1
- net P4_EN: now also TP901.1; no longer SW1.1
- net LED_DATA renamed LED_DIN
- new net BTN_HOME: SW1.1
- new net BTN_PAIR: SW2.1
Other:
- note added: "COMPUTE (record section 8; SPEC: no RP2350, the P4 LP core emits quadrature). Stamp-P4 + Stamp-AddOn C6 stacked on top (SDIO G42-G48, not castellated). Fixed pins only: VIN (14) from +5V, the stamp ORs it with its own USB-C 5V and makes SOC_3.3V itself; all GND pads. No reset button: CHIP_EN and G35 go to tweezer pads TP901 / TP903 beside GND pad TP902 (stamp has 10k pull-ups). G35 appears on pad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"
- note removed: "COMPUTE (record section 8; SPEC: no RP2350, the P4 LP core emits quadrature). Stamp-P4 + Stamp-AddOn C6 stacked on top (SDIO G42-G48, not castellated). Fixed pins only: VIN (14) from +5V, the stamp ORs it with its own USB-C 5V and makes SOC_3.3V itself; all GND pads; CHIP_EN + G35 buttons (stamp has 10k pull-ups). G35 appears on pads 36 AND 48 in M5's own symbol and schematic: both wired to P4_BO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"
