File: flagship/ossm-flagship.kicad_sch (KiCad schematic)
At the start: 0 parts

Commit message: flagship: flatten the schematic to one wired A1 sheet (input left, P4 middle, outputs right, section boxes, notes panel); provisional P4 pin map; connectors placed
Sub-sheet deletion: the root sheet has no (sheet) entries left and no .kicad_* or .md file references the seven sub-sheet files. Netlist compared against the hierarchical design: every pre-existing pin keeps its connections; the only changes are the new P4 pin assignments, the I2C pin swap, pad 48 no-connect, the button pin order, and the new connectors.
Parts:
- added C1, C2, C5, C6: 100u 63V EEH-ZA1J101P, Capacitor_SMD:CP_Elec_10x10.5, symbol Device:C_Polarized
- added C101, C102, C103, C104, C201, C202, C203, C204, C3, C301, C302, C303, C304, C4: 2.2u 100V GRM32ER72A225KA35L, Capacitor_SMD:C_1210_3225Metric, symbol Device:C
- added C105: 5.6n, Capacitor_SMD:C_0805_2012Metric, symbol Device:C
- added C106, C206, C306: DNP, Capacitor_SMD:C_0805_2012Metric, symbol Device:C
- added C107, C207, C307: 0.1u, Capacitor_SMD:C_0805_2012Metric, symbol Device:C
- added C108, C109, C110, C111: 22u 25V, Capacitor_SMD:C_1210_3225Metric, symbol Device:C
- added C13, C14, C601, C602, C802: 100n, Capacitor_SMD:C_0805_2012Metric, symbol Device:C
- added C205, C305: 6.8n, Capacitor_SMD:C_0805_2012Metric, symbol Device:C
- added C208, C209, C210, C308, C309, C310: 47u 10V, Capacitor_SMD:C_1210_3225Metric, symbol Device:C
- added C401: 1u 25V, Capacitor_SMD:C_0805_2012Metric, symbol Device:C
- added C402: 680n 25V, Capacitor_SMD:C_0805_2012Metric, symbol Device:C
- added C501: 1n, Capacitor_SMD:C_0805_2012Metric, symbol Device:C
- added C502: 100n 50V, Capacitor_SMD:C_0805_2012Metric, symbol Device:C
- added C801: 22n 100V, Capacitor_SMD:C_0805_2012Metric, symbol Device:C
- added C803: 100n 100V, Capacitor_SMD:C_1206_3216Metric, symbol Device:C
- added D2, D3, D4: B560C, Diode_SMD:D_SMC, symbol Device:D_Schottky
- added D401: SMBJ48CA, Diode_SMD:D_SMB, symbol Device:D_TVS
- added D5: STATUS_RGB, LED_SMD:LED_WS2812B_PLCC4_5.0x5.0mm_P3.2mm, symbol LED:WS2812B
- added D501: SMBJ48A, Diode_SMD:D_SMB, symbol Device:D_TVS
- added D502: AMBER_CLAMP, LED_SMD:LED_0805_2012Metric, symbol Device:LED
- added D503: SS310, Diode_SMD:D_SMA, symbol Device:D_Schottky
- added D6: RED_FAULT, LED_SMD:LED_1206_3216Metric, symbol Device:LED
- added D601: SM712, flagship:SOT-23-3_L3.0-W1.7-P0.95-LS2.9-BR, symbol flagship:SM712.TCT
- added D801: SMBJ45CA, Diode_SMD:D_SMB, symbol Device:D_TVS
- added D802, D803: BZT52C15, Diode_SMD:D_SOD-123, symbol Device:D_Zener
- added F1: 15A 453 soldered, Fuse:Fuse_Littelfuse-NANO2-451_453, symbol Device:Fuse
- added J1: BUS_IN XT30, flagship:CONN-TH_XT30PW-M, symbol Connector_Generic:Conn_01x02
- added J2: MOTOR XT30, flagship:CONN-TH_XT30PW-M, symbol Connector_Generic:Conn_01x02
- added J3: EXT_SHUNT XT30, flagship:CONN-TH_XT30PW-M, symbol Connector_Generic:Conn_01x02
- added J4: MOTION GH4, Connector_JST:JST_GH_SM04B-GHS-TB_1x04-1MP_P1.25mm_Horizontal, symbol Connector_Generic:Conn_01x04
- added J5: COMMS GH6, Connector_JST:JST_GH_SM06B-GHS-TB_1x06-1MP_P1.25mm_Horizontal, symbol Connector_Generic:Conn_01x06
- added J6: FAN GH4, Connector_JST:JST_GH_SM04B-GHS-TB_1x04-1MP_P1.25mm_Horizontal, symbol Connector_Generic:Conn_01x04
- added J7: THERM GH2, Connector_JST:JST_GH_SM02B-GHS-TB_1x02-1MP_P1.25mm_Horizontal, symbol Connector_Generic:Conn_01x02
- added JP2: FAN 12V default | cut+bridge 5V, Jumper:SolderJumper-3_P1.3mm_Bridged12_RoundedPad1.0x1.5mm_NumberLabels, symbol Jumper:SolderJumper_3_Bridged12
- added JP501: CUT=EXT ONLY, symbol Jumper:SolderJumper_2_Bridged
- added L1: 18u Isat>=7.5A, symbol Device:L
- added L2: 10u Isat>=7.5A, symbol Device:L
- added L3: 6.8u Isat>=7.5A, symbol Device:L
- added Q1, Q2, Q401, Q402, Q501: PSMN3R7-100BSE, Package_TO_SOT_SMD:TO-263-2, symbol flagship:Q_NMOS_D2PAK
- added Q403: DMN10H220L, Package_TO_SOT_SMD:SOT-23, symbol flagship:Q_NMOS_SOT23
- added Q404: MMBT3904, Package_TO_SOT_SMD:SOT-23, symbol Transistor_BJT:MMBT3904
- added Q701: 2N7002, Package_TO_SOT_SMD:SOT-23, symbol Transistor_FET:2N7002
- added R1, R401: 2m CSS2H-2512K-2L00F, flagship:R_2512_Shunt_PseudoKelvin, symbol Device:R_Shunt
- added R101, R201, R301: 887k, Resistor_SMD:R_0805_2012Metric, symbol Device:R
- added R102, R202, R302: 53.6k, Resistor_SMD:R_0805_2012Metric, symbol Device:R
- added R103, R203, R303: 243k, Resistor_SMD:R_0805_2012Metric, symbol Device:R
- added R104: 21.5k, Resistor_SMD:R_0805_2012Metric, symbol Device:R
- added R105: 140k, Resistor_SMD:R_0805_2012Metric, symbol Device:R
- added R106, R17, R18, R206, R26, R28, R306, R411, R502, R504, R507, R512, R601, R804, R806: 10k, Resistor_SMD:R_0805_2012Metric, symbol Device:R
- added R2: 1m WSK12161L000FEA, flagship:R_Shunt_Vishay_WSK1216_Kelvin, symbol Device:R_Shunt
- added R20, R21, R27, R29: 1k, Resistor_SMD:R_0805_2012Metric, symbol Device:R
- added R204: 15.8k, Resistor_SMD:R_0805_2012Metric, symbol Device:R
- added R205: 52.3k, Resistor_SMD:R_0805_2012Metric, symbol Device:R
- added R23: 120R DNP, Resistor_SMD:R_0805_2012Metric, symbol Device:R
- added R24, R25: 4.7k, Resistor_SMD:R_0805_2012Metric, symbol Device:R
- added R30: 27k, Resistor_SMD:R_1206_3216Metric, symbol Device:R
- added R304: 13.7k, Resistor_SMD:R_0805_2012Metric, symbol Device:R
- added R305: 31.6k, Resistor_SMD:R_0805_2012Metric, symbol Device:R
- added R402: 100R, Resistor_SMD:R_0805_2012Metric, symbol Device:R
- added R403: 3.4k, Resistor_SMD:R_0805_2012Metric, symbol Device:R
- added R404: 39.2k, Resistor_SMD:R_0805_2012Metric, symbol Device:R
- added R405, R409, R410, R701: 100k, Resistor_SMD:R_0805_2012Metric, symbol Device:R
- added R406: 8.25k, Resistor_SMD:R_0805_2012Metric, symbol Device:R
- added R407: 470k, Resistor_SMD:R_1206_3216Metric, symbol Device:R
- added R408: 24.9k, Resistor_SMD:R_0805_2012Metric, symbol Device:R
- added R412: 100R, Resistor_SMD:R_2512_6332Metric, symbol Device:R
- added R501: 348k, Resistor_SMD:R_1206_3216Metric, symbol Device:R
- added R503: 3.01M, Resistor_SMD:R_0805_2012Metric, symbol Device:R
- added R505, R801: 10R, Resistor_SMD:R_0805_2012Metric, symbol Device:R
- added R508: 3.3k, Resistor_SMD:R_0805_2012Metric, symbol Device:R
- added R509, R510, R511: 24R D2TO35M, Package_TO_SOT_SMD:TO-263-2, symbol flagship:R_D2PAK_TAB
- added R513: 2.2k, Resistor_SMD:R_0805_2012Metric, symbol Device:R
- added R802: 374k, Resistor_SMD:R_1206_3216Metric, symbol Device:R
- added R803: 15k, Resistor_SMD:R_0805_2012Metric, symbol Device:R
- added R805: 402k, Resistor_SMD:R_1206_3216Metric, symbol Device:R
- added SW1: HOME (hold: RESET), symbol Switch:SW_Push
- added SW2: PAIR (held at power-on: AP), symbol Switch:SW_Push
- added TH501: 10k NCP18XH103F03RB, Resistor_SMD:R_0603_1608Metric, symbol Device:Thermistor_NTC
- added TP901: EN, TestPoint:TestPoint_Pad_D1.5mm, symbol Connector:TestPoint
- added TP902: GND, TestPoint:TestPoint_Pad_D1.5mm, symbol Connector:TestPoint
- added TP903: BOOT, TestPoint:TestPoint_Pad_D1.5mm, symbol Connector:TestPoint
- added U1: LTC4364IS-1, flagship:SOIC-16_L9.9-W3.9-P1.27-LS6.0-BL-1, symbol flagship:LTC4364IS-2#PBF
- added U10: 74AHCT125, Package_SO:TSSOP-14_4.4x5mm_P0.65mm, symbol 74xx:74AHCT125
- added U11: INA228, flagship:VSSOP-10_L3.0-W3.0-P0.50-LS4.9-BL, symbol flagship:INA228AIDGSR
- added U2: TPS48111, flagship:VSSOP-20_19P-L5.0-W3.0-P0.50-LS5.0-BL_PE16, symbol flagship:TPS48111LQDGXRQ1
- added U3: TLV1805, flagship:TSOT-23-6_L2.9-W1.6-P0.95-LS2.8-BL, symbol flagship:TLV1805DBVR
- added U4: TLV431, flagship:SOT-23-3_L2.9-W1.3-P1.90-LS2.4-BR, symbol flagship:TLV431AIDBZR
- added U5: TPS54560B 12V, flagship:POWERPAD-SO-8_L4.9-W3.9-P1.27-LS6.0-BL-EP, symbol flagship:TPS54560BDDAR
- added U6: TPS54560B 5V, flagship:POWERPAD-SO-8_L4.9-W3.9-P1.27-LS6.0-BL-EP, symbol flagship:TPS54560BDDAR
- added U7: TPS54560B 3V3, flagship:POWERPAD-SO-8_L4.9-W3.9-P1.27-LS6.0-BL-EP, symbol flagship:TPS54560BDDAR
- added U8: Stamp-P4, flagship:Stamp-P4, symbol m5stack:Stamp-P4
- added U9: THVD1450, flagship:SOIC-8_L4.9-W3.9-P1.27-LS6.0-BL, symbol flagship:THVD1450DR
Connections:
- new net: D601.2 (A1), J5.3 (Pin_3), R23.2, U9.6 (A)
- new net: J5.5 (Pin_5), R17.2, R20.2
- new net: J5.6 (Pin_6), R18.2, R21.2
- new net: C307.1, U7.1 (BOOT)
- new net: C307.2, D4.1 (K), L3.1, U7.8 (SW)
- new net: C306.1, R304.1, U7.6 (COMP)
- new net: R512.2, TH501.1, U8.25 (G18_ADC1)
- new net: R503.1, R505.2, U3.1 (OUT)
- new net: C501.1, R501.2, R502.1, R503.2, U3.4 (+IN)
- new net: R803.2, R804.1, U1.11 (OV)
- new net: D501.1 (A1), D503.2 (A), J3.2 (Pin_2), JP501.1 (A), Q501.2 (D)
- new net: C207.1, U6.1 (BOOT)
- new net: R201.2, R202.1, U6.3 (EN)
- new net: R203.1, U6.4 (RT/CLK)
- new net: R205.2, R206.1, U6.5 (FB)
- new net: C206.1, R204.1, U6.6 (COMP)
- new net: C207.2, D3.1 (K), L2.1, U6.8 (SW)
- new net: J6.3 (Pin_3), R28.2, R29.2
- new net: R504.1, U3.3 (-IN), U4.1 (REF), U4.2 (C)
- new net: J6.2 (Pin_2), JP2.2 (C)
- new net: J6.4 (Pin_4), Q701.3 (D)
- new net: R1.1, R2.4, R805.1
- new net: R805.2, R806.1, U1.16 (FB)
- new net: JP501.2 (B), R509.3, R510.3, R511.3
- new net: J7.1 (Pin_1), R26.2, R27.2
- new net: R29.1, U8.18 (LPG6)
- new net: Q1.1 (G), R801.1
- new net: D802.2 (A), D803.2 (A), Q1.3 (S), Q2.3 (S), U1.5 (SOURCE)
- new net: D5.4 (DIN), U10.8
- new net: R601.1, U10.9, U8.37 (LPG2)
- new net: Q401.1 (G), Q402.1 (G), U2.14 (PD), U2.15 (PU)
- new net: C401.1, Q401.3 (S), Q402.3 (S), Q403.2 (S), U2.13 (SRC)
- new net: C801.1, D802.1 (K), R801.2, U1.6 (HGATE)
- new net: R406.1, U2.7 (IMON), U8.24 (G19_ADC1)
- new net: Q501.1 (G), R505.1, R507.1, R513.2
- new net: Q701.1 (G), R701.1, U8.29 (LPG13)
- new net: U10.5, U8.35 (LPG5)
- new net: J4.3 (Pin_3), U10.6
- new net: R303.1, U7.4 (RT/CLK)
- new net: R101.2, R102.1, U5.3 (EN)
- new net: C107.1, U5.1 (BOOT)
- new net: C107.2, D2.1 (K), L1.1, U5.8 (SW)
- new net: D6.1 (K), U1.13 (~{FLT})
- new net: D6.2 (A), R30.1
- new net: Q403.3 (D), R412.2
- new net: R24.2, U11.4 (SDA), U8.6 (LPG9)
- new net: C305.1, R304.2
- new net: C14.1, R27.1, U8.27 (G16_ADC1)
- new net: TP901.1, U8.34 (CHIP_EN)
- new net: Q401.2 (D), R401.1
- new net: R401.2, U2.17 (CS-)
- new net: R401.3, R402.1
- new net: U8.46 (G32_RMII_CLK), U9.1 (R)
- new net: U8.49 (G41_RMII_TXD0), U9.2 (~{RE}), U9.3 (DE)
- new net: U8.50 (G33_RMII_TXEN), U9.4 (D)
- new net: C401.2, U2.12 (BST)
- new net: SW1.2, U8.12 (G49_ADC2)
- new net: R407.2, R408.1, U11.3 (ALERT), U2.1 (EN/UVLO), U8.20 (G23_ADC1)
- new net: R301.2, R302.1, U7.3 (EN)
- new net: R305.2, R306.1, U7.5 (FB)
- new net: R404.1, U2.8 (IWRN)
- new net: F1.1, J1.1 (Pin_1)
- new net: R409.1, U2.3 (INP), U8.22 (G21_ADC1)
- new net: J4.1 (Pin_1), U10.3
- new net: C106.1, R104.1, U5.6 (COMP)
- new net: C105.1, R104.2
- new net: D502.2 (A), R513.1
- new net: C205.1, R204.2
- new net: Q404.1 (B), Q404.3 (C), U2.10 (DIODE)
- new net: R402.2, U2.18 (CS+)
- new net: R403.2, U2.19 (ISCP)
- new net: R410.1, U2.2 (INP_G), U8.21 (G22_ADC1)
- new net: R411.1, U2.4 (~{FLT_T}), U2.5 (~{FLT_I}), U8.23 (G20_ADC1)
- new net: C402.1, R405.1, U2.9 (TMR)
- new net: TP903.1, U8.36 (G35_BOOT_RMII_TXD1)
- new net: R20.1, U8.51 (G31_RMII_MDC)
- new net: D803.1 (K), Q2.1 (G), U1.4 (DGATE)
- new net: Q2.2 (D), R1.4
- new net: R105.2, R106.1, U5.5 (FB)
- new net: R103.1, U5.4 (RT/CLK)
- new net: C802.1, U1.15 (TMR)
- new net: U10.2, U8.45 (LPG3)
- new net: R1.2, U1.1 (OUT)
- new net: R802.2, R803.1, U1.10 (UV)
- new net: R1.3, U1.2 (SENSE)
- new net: R507.2, R508.1, U8.26 (G17_ADC1)
- new net: R25.2, U11.5 (SCL), U8.4 (LPG11)
- new net: R2.3, U11.10 (IN+)
- new net: R2.2, U11.9 (IN-)
- new net: SW2.2, U8.16 (LPG4)
- new net: R21.1, U8.52 (G28_RMII_RXDV)
- new net +12V: C108.1, C109.1, C110.1, C111.1, C502.1, JP2.1 (A), L1.2, R105.1, R504.2, U3.6 (V+)
- new net +3V3_ACC: C308.1, C309.1, C310.1, L3.2, R305.1
- new net +3V3_SYS: C13.1, C601.1, D601.1 (A1), J5.4 (Pin_4), R17.1, R18.1, R23.1, R24.1, R25.1, R26.1, R28.1, R411.2, R512.1, U11.6 (VS), U8.28 (SOC_3.3V), U9.7 (B), U9.8 (VCC)
- new net +5V: C208.1, C209.1, C210.1, JP2.3 (B), L2.2, R205.1, U8.14 (VIN)
- new net +5V_SYS: C602.1, D5.1 (VDD), J5.1 (Pin_1), U10.13, U10.14 (VCC), U8.39 (SYS_5V)
- new net +BUS: C1.1, C101.1, C102.1, C103.1, C104.1, C2.1, C201.1, C202.1, C203.1, C204.1, C3.1, C301.1, C302.1, C303.1, C304.1, C4.1, C5.1, C6.1, D503.1 (K), J3.1 (Pin_1), R101.1, R2.1, R201.1, R301.1, R401.4, R403.1, R407.1, R412.1, R501.1, R509.1, R510.1, R511.1, U11.8 (VBUS), U2.20 (VS), U5.2 (VIN), U6.2 (VIN), U7.2 (VIN)
- new net GND: C1.2, C101.2, C102.2, C103.2, C104.2, C105.2, C106.2, C108.2, C109.2, C110.2, C111.2, C13.2, C14.2, C2.2, C201.2, C202.2, C203.2, C204.2, C205.2, C206.2, C208.2, C209.2, C210.2, C3.2, C301.2, C302.2, C303.2, C304.2, C305.2, C306.2, C308.2, C309.2, C310.2, C4.2, C402.2, C5.2, C501.2, C502.2, C6.2, C601.2, C602.2, C801.2, C802.2, C803.2, D2.2 (A), D3.2 (A), D4.2 (A), D401.1 (A1), D5.3 (VSS), D501.2 (A2), D502.1 (K), D601.3 (K), D801.1 (A1), J1.2 (Pin_2), J2.2 (Pin_2), J4.2 (Pin_2), J4.4 (Pin_4), J5.2 (Pin_2), J6.1 (Pin_1), J7.2 (Pin_2), Q404.2 (E), Q501.3 (S), Q701.2 (S), R102.2, R103.2, R106.2, R202.2, R203.2, R206.2, R302.2, R303.2, R306.2, R404.2, R405.2, R406.2, R408.2, R409.2, R410.2, R502.2, R508.2, R509.2 (TAB), R510.2 (TAB), R511.2 (TAB), R601.2, R701.2, R804.2, R806.2, SW1.1, SW2.1, TH501.2, TP902.1, U1.12 (GND), U10.1, U10.10, U10.12, U10.4, U10.7 (GND), U11.1 (A1), U11.2 (A0), U11.7 (GND), U2.6 (GND), U3.2 (V-), U3.5 (SHDN), U4.3 (A), U5.7 (GND), U5.9 (EP), U6.7 (GND), U6.9 (EP), U7.7 (GND), U7.9 (EP), U8.13 (GND), U8.38 (GND), U8.42 (GND), U8.56 (GND), U8.59 (GND), U8.62 (GND), U8.65 (GND), U9.5 (GND)
- new net MOTOR_V+: D401.2 (A2), J2.1 (Pin_1), Q402.2 (D)
- new net PRE_G: Q403.1 (G), U2.11 (G)
- new net VIN_RAW: C803.1, D801.2 (A2), F1.2, Q1.2 (D), R30.2, R802.1, U1.8 (VCC)
- no-connect marks 0 -> 6
Other:
- removed sheet Compute
- removed sheet Drive IO
- removed sheet Input protection
- removed sheet Motor switch
- removed sheet Rails
- removed sheet Regen shunt
- removed sheet Sensing
- note added: "BUCK RAILS"
- note added: "COMPUTE (STAMP-P4)"
- note added: "COMPUTE (record section 8; SPEC: no RP2350, the P4 LP core emits quadrature). Stamp-P4 + Stamp-AddOn C6 stacked on top (SDIO G42-G48, not castellated). Fixed pins only: VIN (14) from +5V, the stamp ORs it with its own USB-C 5V and makes SOC_3.3V itself; all GND pads. No reset button: CHIP_EN and G35 go to tweezer pads TP901 / TP903 beside GND pad TP902 (stamp has 10k pull-ups). G35 appears on pad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"
- note added: "DRIVE INTERFACE"
- note added: "DRIVE IO (record sections 11-12; SPEC: 3.3 V RS485 non-isolated, quadrature via 74AHCT125, JST GH signals). Connectors are the operator's: every off-board net ends in a named label (DRV_*, and +5V_SYS for the drive's 485_5V on comms pin 10; PU-/DIR-/COM are GND). U9 THVD1450 on a P4 UART in RS485 half-duplex mode, DE and /RE tied. R23 termination fitted- not-populated. D601 SM712 (-7/+12 V RS485 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"
- note added: "FAN + THERMISTOR"
- note added: "INPUT PROTECTION"
- note added: "INPUT PROTECTION (record section 3). Self-acting: nothing depends on firmware or a rail it protects. LTC4364-1 datasheet Figure 1 topology. F1 Nano2 453 15 A soldered: dead-short backstop. D801 SMBJ45CA (bidirectional: survives a reversed supply) clamps the hot-plug ring. Q1 hot-swap FET on HGATE, Q2 ideal-diode FET on DGATE, common SOURCE: reverse polarity AND reverse current blocked, so the reg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"
- note added: "MOTOR SWITCH"
- note added: "MOTOR SWITCH (record section 4). TPS48111 datasheet Figure 9-14 topology: back-to-back N-FETs, common source, pre-charge through Q403 and Q402's body diode. Open = open both ways: back-drive never reaches the board, so the regen shunt sizes for the powered 6.8 W case. FETs Q401/Q402: 100 V (58.6 V back-EMF), D2PAK class; TODO pick part. R401 2 mOhm: 30 mV at 15 A. OC R404 39.2k = 15.2 A for 10 ms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"
- note added: "NOTES"
- note added: "POWER MONITOR (INA228)"
- note added: "RAILS (record section 10: independent bucks from +BUS). TPS54560B x3, one layout three times; values from the datasheet's own design procedure (SLVSF00 section 8.2). Design inputs: VIN 20-48 V (48 = supply OVP ceiling, covers the ~45 V clamp; part rated 60 V), 4 A per rail, 400 kHz, half-load step held within 4 %. fsw 400 kHz: RT 243k. Worst on-time 3.3 V at 48 V = 205 ns vs 135 ns minimum. UVLO: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"
- note added: "REGEN CLAMP"
- note added: "REGEN SHUNT (record section 5). Self-acting clamp, no firmware: U3 compares the divided bus to U4's 1.24 V; R503 hysteresis. R501/R502/R503 348k/10k/3.01M: ON 44.5 V, OFF 43.2 V (1.4 V hysteresis, the OSSM alt board's value). Legal above the GST360A36's 37.8 V worst OVP only because the input section blocks reverse current. R509 || R510 || R511: Vishay D2TO35M 24R each = 8R (multi-pulse rated; el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"
- note added: "SENSING (record sections 10, 12). U11 INA228 on the R2 Kelvin taps (Input sheet): route INA_SENSE_P/N as a tight pair, INA beside the shunt, away from switch nodes. 1 mOhm: 10 mV at 10 A in the +-163.84 mV range. Die temperature = board temperature. A0/A1 = GND (0x40). INA_ALERT_N (open drain) is also the motor-switch EN: over-current / power / temperature limits cut the motor with no MCU. R24/R2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"

Commit message: flagship: tidy every schematic section (compact layouts, no overlapping text, grounds bused, PRE_G drawn as a wire); netlist verified identical
Eight per-section passes applied one at a time to the flat sheet, each checked against the pre-tidy netlist (identical after every step). ERC: only the spare Stamp-P4 pins remain unconnected.
Connections:
- net +3V3_SYS: no longer D601.1 (A1), J5.4 (Pin_4), R23.1, U9.7 (B)
- net PRE_G: no longer names the net of Q403.1 (G), U2.11 (G)
- new net: D601.1 (A1), J5.4 (Pin_4), R23.1, U9.7 (B)
- no-connect marks 6 -> 7
Other:
- moved on the sheet: C101, C102, C103, C104, C105, C106, C107, C108, C109, C110, C111, C13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

Commit message: flagship: J8 firmware probe header (QUAD_A, GND, DBG, QUAD_B) + R602 1k on spare G50 for a DBG trigger pin
Parts:
- added J8: PROBE 1x4 2.54, Connector_PinHeader_2.54mm:PinHeader_1x04_P2.54mm_Vertical, symbol Connector_Generic:Conn_01x04
- added R602: 1k, Resistor_SMD:R_0805_2012Metric, symbol Device:R
Connections:
- net GND: now also J8.2 (Pin_2)
- net at U10.5, U8.35 (LPG5): now also J8.4 (Pin_4)
- net at U10.2, U8.45 (LPG3): now also J8.1 (Pin_1)
- net at U8.10 (G50_ADC2): now also R602.2
- new net DBG: J8.3 (Pin_3), R602.1
