File: flagship/ossm-flagship.kicad_sch (KiCad schematic)
At the start: 165 parts, among them J1 BUS_IN XT30, J2 MOTOR XT30, J3 EXT_SHUNT XT30, J4 MOTION GH4, J5 COMMS GH6, J6 FAN GH4, J7 THERM GH2, J8 PROBE 1x4 2.54, Q1 PSMN3R7-100BSE, Q2 PSMN3R7-100BSE, Q401 PSMN3R7-100BSE, Q402 PSMN3R7-100BSE, Q403 DMN10H220L, Q404 MMBT3904, Q501 PSMN3R7-100BSE, Q701 2N7002, SW1 HOME (hold: RESET), SW2 PAIR (held at power-on: AP), U1 LTC4364IS-1, U10 74AHCT125, U11 INA228, U2 TPS48111, U3 TLV1805, U4 TLV431, U5 TPS54560B 12V, U6 TPS54560B 5V, U7 TPS54560B 3V3, U8 Stamp-P4, U9 THVD1450

Commit message: flagship: power FETs -> IPB042N10N3G x5 (C802 timer 22 nF C0G keeps Q1 in SOA), bulk -> 4 x EEH-ZA1J820P 82 uF 63 V; BOM ~$89/board at 5, ~$65 at 40
Parts:
- C1, C2, C5, C6: value 100u 63V EEH-ZA1J101P -> 82u 63V EEH-ZA1J820P
- C802: value 100n -> 22n C0G
- Q1, Q2, Q401, Q402, Q501: value PSMN3R7-100BSE -> IPB042N10N3G
Other:
- note added: "MOTOR SWITCH (record section 4). TPS48111 datasheet Figure 9-14 topology: back-to-back N-FETs, common source, pre-charge through Q403 and Q402's body diode. Open = open both ways: back-drive never reaches the board, so the regen shunt sizes for the powered 6.8 W case. FETs Q401/Q402: 100 V (58.6 V back-EMF), IPB042N10N3G (D2PAK). R401 2 mOhm: 30 mV at 15 A. OC R404 39.2k = 15.2 A for 10 ms (C402 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"
- note removed: "MOTOR SWITCH (record section 4). TPS48111 datasheet Figure 9-14 topology: back-to-back N-FETs, common source, pre-charge through Q403 and Q402's body diode. Open = open both ways: back-drive never reaches the board, so the regen shunt sizes for the powered 6.8 W case. FETs Q401/Q402: 100 V (58.6 V back-EMF), D2PAK class; TODO pick part. R401 2 mOhm: 30 mV at 15 A. OC R404 39.2k = 15.2 A for 10 ms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"

Commit message: flagship: bus-powered OVP trip (51 V zener + NPN on the TPS48111 EN node) cuts motor power on bus overvoltage, no firmware needed
Parts:
- added D402: BZT52C51, Diode_SMD:D_SOD-123, symbol Device:D_Zener
- added Q405: MMBT3904, Package_TO_SOT_SMD:SOT-23, symbol Transistor_BJT:MMBT3904
- added R413, R414: 10k, Resistor_SMD:R_0805_2012Metric, symbol Device:R
Connections:
- net +BUS: now also D402.1 (K)
- net GND: now also Q405.2 (E), R414.1
- net at R407.2, R408.1, U11.3 (ALERT)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: now also Q405.3 (C)
- new net: Q405.1 (B), R413.2, R414.2
- new net: D402.2 (A), R413.1

Commit message: flagship: 24-36 V input (R408 30.1k: motor UVLO 19.6/18.4 V; R803 17.8k: LTC4364 UV 18.1 V); motor pairing recorded; C401 note corrected to 1u
Parts:
- R408: value 24.9k -> 30.1k
- R803: value 15k -> 17.8k
Other:
- note added: "MOTOR SWITCH (record section 4). TPS48111 datasheet Figure 9-14 topology: back-to- back N-FETs, common source, pre-charge through Q403 and Q402's body diode. Open = open both ways: back-drive never reaches the board, so the regen shunt sizes for the powered 6.8 W case. FETs Q401/Q402: 100 V (58.6 V back-EMF), IPB042N10N3G (D2PAK). R401 2 mOhm: 30 mV at 15 A. OC R404 39.2k = 15.2 A for 10 ms (C402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"
- note removed: "MOTOR SWITCH (record section 4). TPS48111 datasheet Figure 9-14 topology: back-to-back N-FETs, common source, pre-charge through Q403 and Q402's body diode. Open = open both ways: back-drive never reaches the board, so the regen shunt sizes for the powered 6.8 W case. FETs Q401/Q402: 100 V (58.6 V back-EMF), IPB042N10N3G (D2PAK). R401 2 mOhm: 30 mV at 15 A. OC R404 39.2k = 15.2 A for 10 ms (C402 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"
Changed lines of the file:
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@@
 		)
 	)
-	(text "INPUT PROTECTION (record section 3). Self-acting: nothing depends on firmware or a\n  rail it protects. LTC4364-1 datasheet Figure 1 topology.\nF1 Nano2 453 15 A soldered: dead-short backstop. D801 SMBJ45CA (bidirectional:\n  survives a reversed supply) clamps the hot-plug ring.\nQ1 hot-swap FET on HGATE, Q2 ideal-diode FET on DGATE, common SOURCE: reverse\n  polarity AND reverse current blocked, so the regen clamp may sit at 44.5 V.\nR1 2 mOhm CSS2H, pseudo-Kelvin (SENSE and OUT on the inner-edge sense pads): 50 mV =\n  25 A limit (25 mV = 12.5 A folded back into a short). C802 22n C0G: ~0.23 ms in a\n  dead short (36 V x 12.5 A = 450 W in Q1), ~2.4 ms on a mild overload.\nC801 22n on HGATE: ~40 ms power-up ramp, ~0.4 A inrush into ~480 uF (4 x 82 uF bulk\n  + the drive's 150 uF + ceramics): the current limit and timer never engage at\n  start.\nR805/R806 402k/10k: output clamp 51.5 V, ABOVE the 44.5 V regen clamp so regen is\n  never read as an input surge (LTC4364-1 would latch).\nR802/R803/R804 374k/15k/10k: UV 20 V, OV 50 V. D802/D803 15 V gate zeners\n  (datasheet: required at >= 24 V). SHDN and ENOUT unused.\nLATCH-OFF (-1): a fault kills every rail; D6 + R30 27k from VIN_RAW light on FLT\n  with the board dark (FLT sinks <= 2 mA: 1.3 mA at 36 V). Power-cycle to clear.\nQ1/Q2 IPB042N10N3G: SOA ~55 A at 36 V for 0.2 ms (25 C); worst case (OUT just above\n  2.5 V, ~27 A at ~33 V, ~0.25 ms) keeps ~1.75x cold, ~1.35x hot. R2 = INA228 shunt,\n  WSK1216 true 4-terminal Kelvin."
+	(text "INPUT PROTECTION (record section 3). Self-acting: nothing depends on firmware or a\n  rail it protects. LTC4364-1 datasheet Figure 1 topology.\nF1 Nano2 453 15 A soldered: dead-short backstop. D801 SMBJ45CA (bidirectional:\n  survives a reversed supply) clamps the hot-plug ring.\nQ1 hot-swap FET on HGATE, Q2 ideal-diode FET on DGATE, common SOURCE: reverse\n  polarity AND reverse current blocked, so the regen clamp may sit at 44.5 V.\nR1 2 mOhm CSS2H, pseudo-Kelvin (SENSE and OUT on the inner-edge sense pads): 50 mV =\n  25 A limit (25 mV = 12.5 A folded back into a short). C802 22n C0G: ~0.23 ms in a\n  dead short (36 V x 12.5 A = 450 W in Q1), ~2.4 ms on a mild overload.\nC801 22n on HGATE: ~40 ms power-up ramp, ~0.4 A inrush into ~480 uF (4 x 82 uF bulk\n  + the drive's 150 uF + ceramics): the current limit and timer never engage at\n  start.\nR805/R806 402k/10k: output clamp 51.5 V, ABOVE the 44.5 V regen clamp so regen is\n  never read as an input surge (LTC4364-1 would latch).\nR802/R803/R804 374k/17.8k/10k: UV 18.1 V, OV 50.2 V (24-36 V input). D802/D803 15 V\n  gate zeners (datasheet: required at >= 24 V). SHDN and ENOUT unused.\nLATCH-OFF (-1): a fault kills every rail; D6 + R30 27k from VIN_RAW light on FLT\n  with the board dark (FLT sinks <= 2 mA: 1.3 mA at 36 V). Power-cycle to clear.\nQ1/Q2 IPB042N10N3G: SOA ~55 A at 36 V for 0.2 ms (25 C); worst case (OUT just above\n  2.5 V, ~27 A at ~33 V, ~0.25 ms) keeps ~1.75x cold, ~1.35x hot. R2 = INA228 shunt,\n  WSK1216 true 4-terminal Kelvin."
 		(exclude_from_sim no)
 		(at 474.98 196.85 0)
@@
 		)
 	)
-	(text "MOTOR SWITCH (record section 4). TPS48111 datasheet Figure 9-14 topology:\n  back-to-back N-FETs, common source, pre-charge through Q403 and Q402's body\n  diode.\nOpen = open both ways: back-drive never reaches the board, so the regen shunt\n  sizes for the powered 6.8 W case.  FETs Q401/Q402: 100 V (58.6 V back-EMF),\n  IPB042N10N3G (D2PAK).\nR401 2 mOhm: 30 mV at 15 A. OC R404 39.2k = 15.2 A for 10 ms (C402 680n, R405\n  100k = LATCH-OFF; firmware re-arms by toggling MOTOR_EN). SC R403 3.4k = 30\n  A in 1.2 us.\nIMON R406 8.25k: 3.0 V at 20 A into an ADC1 pin.  CBST C401 470n.  UVLO\n  R407/R408 470k/24.9k: on above ~23 V.  Q404 sits beside Q401/Q402 in layout:\n  150 C cutoff.\nMOTOR_EN floats during P4 boot: R409 pulldown + internal pulldown = off.\n  INA_ALERT_N (open drain) pulls EN low: INA228 limits cut the motor with no\n  MCU.\nPRE-CHARGE: drive input measured 150 uF (hw-x65). PRECHARGE_EN high ~75 ms\n  (R412 100R, 0.36 A peak, ~0.1 J), then MOTOR_EN high, then PRECHARGE_EN low.\nD401 SMBJ48CA: stands off above the 45 V clamp, clamps under the 100 V FETs;\n  catches the hot-plug ring of the drive's ceramic input."
+	(text "MOTOR SWITCH (record section 4). TPS48111 datasheet Figure 9-14 topology: back-to-\n  back N-FETs, common source, pre-charge through Q403 and Q402's body diode.\nOpen = open both ways: back-drive never reaches the board, so the regen shunt sizes\n  for the powered 6.8 W case.  FETs Q401/Q402: 100 V (58.6 V back-EMF), IPB042N10N3G\n  (D2PAK).\nR401 2 mOhm: 30 mV at 15 A. OC R404 39.2k = 15.2 A for 10 ms (C402 680n, R405 100k =\n  LATCH-OFF; firmware re-arms by toggling MOTOR_EN). SC R403 3.4k = 30 A in 1.2 us.\nIMON R406 8.25k: 3.0 V at 20 A into an ADC1 pin.  CBST C401 1u. UVLO R407/R408\n  470k/30.1k: on 19.6 V, off 18.4 V (24-36 V input; the EN node reads 3.31 V at 55\n  V, safe for P4 G23).  Q404 sits beside Q401/Q402 in layout: 150 C cutoff.\nMOTOR_EN floats during P4 boot: R409 pulldown + internal pulldown = off. INA_ALERT_N\n  (open drain) pulls EN low: INA228 limits cut the motor with no MCU.\nPRE-CHARGE: drive input measured 150 uF (hw-x65). PRECHARGE_EN high ~75 ms (R412\n  100R, 0.36 A peak, ~0.1 J), then MOTOR_EN high, then PRECHARGE_EN low.\nD401 SMBJ48CA: stands off above the 45 V clamp, clamps under the 100 V FETs; catches\n  the hot-plug ring of the drive's ceramic input."
 		(exclude_from_sim no)
 		(at 588.01 285.75 0)
@@
 			)
 		)
-		(property "Value" "24.9k"
+		(property "Value" "30.1k"
 			(at 378.46 121.92 0)
 			(show_name no)
@@
 			)
 		)
-		(property "Value" "15k"
+		(property "Value" "17.8k"
 			(at 54.61 121.92 0)
 			(show_name no)

Commit message: flagship: regen bank 24 x 200R anti-surge 2512; fan 3-pin, 5 V default, high-side PWM
Regen: R509-R511 (3 x D2TO35M 24R, unstocked) replaced by R521-R544, 24 x UniOhm
AS122WJ0201T4E 200R 2512 in parallel = 8.33 R (LCSC C2770484, ~$2/board). No tabs,
so the bank no longer touches GND. BOM totals now include it.

Fan: J6 GH4 -> GH3 (1 GND, 2 +V, 3 TACH). Q702 AO3401A high-side on the fan's +V
so the tach ground stays solid; Q701 2N7002 drives its gate through R703 470R
against R702 1k (Vgs -8.2 V on the 12 V setting, under the +-12 V rating).
D701 B5819W flyback. JP2 now defaults to 5 V.

Netlist diffed per pin against the previous baseline: only these changes.
ERC: 29 errors, all unused Stamp-P4 (U8) pins.
Parts:
- removed J6: FAN GH4, Connector_JST:JST_GH_SM04B-GHS-TB_1x04-1MP_P1.25mm_Horizontal, symbol Connector_Generic:Conn_01x04
- removed R509, R510, R511: 24R D2TO35M, Package_TO_SOT_SMD:TO-263-2, symbol flagship:R_D2PAK_TAB
- added D701: B5819W, Diode_SMD:D_SOD-123, symbol Device:D_Schottky
- added J6: FAN GH3, Connector_JST:JST_GH_SM03B-GHS-TB_1x03-1MP_P1.25mm_Horizontal, symbol Connector_Generic:Conn_01x03
- added Q702: AO3401A, Package_TO_SOT_SMD:SOT-23, symbol Transistor_FET:AO3401A
- added R521, R522, R523, R524, R525, R526, R527, R528, R529, R530, R531, R532, R533, R534, R535, R536, R537, R538, R539, R540, R541, R542, R543, R544: 200R AS122WJ0201T4E, Resistor_SMD:R_2512_6332Metric, symbol Device:R
- added R702: 1k, Resistor_SMD:R_0805_2012Metric, symbol Device:R
- added R703: 470R, Resistor_SMD:R_0805_2012Metric, symbol Device:R
- JP2: value FAN 12V default | cut+bridge 5V -> FAN 5V default | cut+bridge 12V
Connections:
- net +12V: now also JP2.3 (B); no longer JP2.1 (A)
- net +5V: now also JP2.1 (A); no longer JP2.3 (B)
- net +BUS: now also R521.1, R522.2, R523.1, R524.2, R525.1, R526.2, R527.1, R528.2, R529.1, R530.2, R531.1, R532.2, R533.1, R534.2, R535.1, R536.2, R537.1, R538.2, R539.1, R540.2, R541.1, R542.2, R543.1, R544.2
- net GND: now also D701.2 (A), J6.1 (Pin_1)
- net at R28.2, R29.2: now also J6.3 (Pin_3)
- net at JP2.2 (C): now also Q702.2 (S), R702.1
- net at Q701.3 (D): now also R703.1
- net at JP501.2 (B): now also R521.2, R522.1, R523.2, R524.1, R525.2, R526.1, R527.2, R528.1, R529.2, R530.1, R531.2, R532.1, R533.2, R534.1, R535.2, R536.1, R537.2, R538.1, R539.2, R540.1, R541.2, R542.1, R543.2, R544.1
- new net: Q702.1 (G), R702.2, R703.2
- new net: D701.1 (K), J6.2 (Pin_2), Q702.3 (D)
Other:
- note added: "R521-R544: 24 x 200R AS122WJ0201T4E (2512, LCSC C2770484), 8.33 R total"
- note added: "REGEN SHUNT (record section 5). Self-acting clamp, no firmware: U3 compares the divided bus to U4's 1.24 V; R503 hysteresis. R501/R502/R503 348k/10k/3.01M: ON 44.5 V, OFF 43.2 V (1.4 V hysteresis, the OSSM alt board's value). Legal above the GST360A36's 37.8 V worst OVP only because the input section blocks reverse current. R521-R544: 24 x 200R UniOhm AS122WJ0201T4E anti-surge 2512 in parallel = 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"
- note removed: "REGEN SHUNT (record section 5). Self-acting clamp, no firmware: U3 compares the divided bus to U4's 1.24 V; R503 hysteresis. R501/R502/R503 348k/10k/3.01M: ON 44.5 V, OFF 43.2 V (1.4 V hysteresis, the OSSM alt board's value). Legal above the GST360A36's 37.8 V worst OVP only because the input section blocks reverse current. R509 || R510 || R511: Vishay D2TO35M 24R each = 8R (multi-pulse rated; el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"
- moved on the sheet: JP2, Q701, R28

Commit message: flagship: fan supply filtered to DC with damping and polyfuse; connector short protection
Fan: L701 100 uH + C701 22 uF after Q702 (D701 freewheels) so the tach is valid
at every speed; R704 1R + C702 100 uF damp the LC (simulated hard-step overshoot
0-6 %, was +60-75 %); F701 0.5 A polyfuse in the fan feed.

Connectors: F601 0.1 A polyfuse on the COMMS 5 V out; R603/R604 180R on the
MOTION pulse outputs; R605/R606 1k on the probe-header taps (J8 moved).

Netlist diffed per pin against the previous baseline: only these changes.
ERC: 29 errors, all unused Stamp-P4 (U8) pins, same as before.
Parts:
- added C701: 22u 25V, Capacitor_SMD:C_1206_3216Metric, symbol Device:C
- added C702: 100u 25V RVT1E101M0607, Capacitor_SMD:CP_Elec_6.3x7.7, symbol Device:C_Polarized
- added F601: 0.1A 1206L010/60NRL, Fuse:Fuse_1206_3216Metric, symbol Device:Polyfuse
- added F701: 0.5A 1206L050/33NR, Fuse:Fuse_1206_3216Metric, symbol Device:Polyfuse
- added L701: 100u SWPA6045S101MT, Inductor_SMD:L_Sunlord_SWPA6045S, symbol Device:L
- added R603, R604: 180R, Resistor_SMD:R_0805_2012Metric, symbol Device:R
- added R605, R606: 1k, Resistor_SMD:R_0805_2012Metric, symbol Device:R
- added R704: 1R, Resistor_SMD:R_1206_3216Metric, symbol Device:R
Connections:
- net +5V_SYS: now also F601.1; no longer J5.1 (Pin_1)
- net GND: now also C701.2, C702.2
- net at U10.5, U8.35 (LPG5): now also R606.1; no longer J8.4 (Pin_4)
- net at U10.6: now also R604.1; no longer J4.3 (Pin_3)
- net at Q702.2 (S), R702.1: now also F701.2; no longer JP2.2 (C)
- net at D701.1 (K), Q702.3 (D): now also L701.1; no longer J6.2 (Pin_2)
- net at J4.1 (Pin_1): now also R603.2; no longer U10.3
- net at U10.2, U8.45 (LPG3): now also R605.1; no longer J8.1 (Pin_1)
- new net: F601.2, J5.1 (Pin_1)
- new net: C701.1, J6.2 (Pin_2), L701.2, R704.1
- new net: J8.4 (Pin_4), R606.2
- new net: C702.1, R704.2
- new net: J4.3 (Pin_3), R604.2
- new net: F701.1, JP2.2 (C)
- new net: R603.1, U10.3
- new net: J8.1 (Pin_1), R605.2
Other:
- note added: "DRIVE IO (record sections 11-12; SPEC: 3.3 V RS485 non-isolated, quadrature via 74AHCT125, JST GH signals). Connectors are the operator's: every off-board net ends in a named label (DRV_*, and +5V_SYS for the drive's 485_5V on comms pin 10; PU-/DIR-/COM are GND). U9 THVD1450 on a P4 UART in RS485 half-duplex mode, DE and /RE tied. R23 termination fitted-not-populated. D601 SM712 (-7/+12 V RS485 E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"
- note removed: "DRIVE IO (record sections 11-12; SPEC: 3.3 V RS485 non-isolated, quadrature via 74AHCT125, JST GH signals). Connectors are the operator's: every off-board net ends in a named label (DRV_*, and +5V_SYS for the drive's 485_5V on comms pin 10; PU-/DIR-/COM are GND). U9 THVD1450 on a P4 UART in RS485 half-duplex mode, DE and /RE tied. R23 termination fitted- not-populated. D601 SM712 (-7/+12 V RS485 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"
- moved on the sheet: J4, J6, J8, JP2

Commit message: flagship: external wired E-stop (COM/NC/NO, hardware trip, unplugged-only single-session bypass)
J9 GH3 with R901/R902 2.2k pull-ups, C901/C902, D901 PESD3V3S2UT. NC open drives
Q901 onto the motor-switch EN wired-OR node (with the bus OVP and INA ALERT): a
hardware stop. NC/NO read on G39/G30 through 1k. Bypass G29 -> Q903 in series
with Q902 (gated by NO open), so only an unplugged cable can be masked; R906
pull-down clears it on every reset. Resolves the SPEC open item.

Netlist diffed per pin against the previous baseline: only additions; U8 pins
31/53/54 leave the unconnected list. ERC: 26 errors, all unused Stamp-P4 pins.
Parts:
- added C901, C902: 100n, Capacitor_SMD:C_0805_2012Metric, symbol Device:C
- added D901: PESD3V3S2UT, Package_TO_SOT_SMD:SOT-23, symbol Device:D_TVS_Dual_AAC
- added J9: ESTOP GH3, Connector_JST:JST_GH_SM03B-GHS-TB_1x03-1MP_P1.25mm_Horizontal, symbol Connector_Generic:Conn_01x03
- added Q901, Q902, Q903: 2N7002, Package_TO_SOT_SMD:SOT-23, symbol Transistor_FET:2N7002
- added R901, R902: 2.2k, Resistor_SMD:R_0805_2012Metric, symbol Device:R
- added R903, R904: 1k, Resistor_SMD:R_0805_2012Metric, symbol Device:R
- added R905, R906: 100k, Resistor_SMD:R_0805_2012Metric, symbol Device:R
Connections:
- net +3V3_SYS: now also R901.1, R902.1
- net GND: now also C901.2, C902.2, D901.3 (common), J9.1 (Pin_1), Q901.2 (S), Q903.2 (S), R906.2
- net at Q405.3 (C), R407.2, R408.1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: now also Q901.3 (D)
- net at U8.31 (G39): now also R903.1
- net at U8.53 (G30_RMII_RXD1): now also R904.1
- net at U8.54 (G29_RMII_RXD0): now also Q903.1 (G), R906.1
- new net: C902.1, D901.2 (A2), J9.3 (Pin_3), Q902.1 (G), R902.2, R904.2
- new net: C901.1, D901.1 (A1), J9.2 (Pin_2), R901.2, R903.2, R905.1
- new net: Q901.1 (G), Q902.3 (D), R905.2
- new net: Q902.2 (S), Q903.3 (D)
Other:
- note added: "EXTERNAL E-STOP"
- note added: "EXTERNAL E-STOP (operator, 2026-09-23). J9 GH3 carries COM / NC / NO of a latching button; COM is GND, R901/R902 2.2k pull NC and NO to 3V3 (~1.5 mA contact wetting), C901/C902 + D901 PESD3V3S2UT at the connector. Hardware stop, no firmware: NC open (pressed OR unplugged) drives Q901 through R905 and pulls the motor-switch EN low, the same wired-OR node as the bus OVP (Q405) and INA ALERT. Firmwa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"

Commit message: flagship: LP pins carry quadrature only (six signals moved to HP GPIOs); budget-build bypass links drawn
Pins: INA228 SDA LPG9->G34, SCL LPG11->G36, LED_DATA LPG2->G26, FAN_PWM
LPG13->G27, FAN_TACH LPG6->G38, BTN_PAIR LPG4->G52; LPG3/LPG5 keep QUAD_A/B and
every other LPG pin is unused. Strap safety per the Stamp-P4 schematic and
ESP32-P4 DS/TRM (SPEC row). DSI GND bus nudged to free the G52 lane.

Links: JP801 (bypasses the LTC4364 stage), JP401 (bypasses the motor switch),
flagship:Link_Wire_15A footprint, DNP and out of the BOM.

Netlist diffed per pin: only the two links and the six pin moves. ERC: 26
errors, all unused Stamp-P4 pins.
Parts:
- added JP401, JP801: BUDGET LINK (open), flagship:Link_Wire_15A, symbol Jumper:Jumper_2_Open
Connections:
- net +BUS: now also JP401.1 (A)
- net MOTOR_V+: now also JP401.2 (B)
- net VIN_RAW: now also JP801.1 (A)
- net at R1.1, R2.4, R805.1: now also JP801.2 (B)
- net at R29.1: now also U8.32 (G38_U0RX); no longer U8.18 (LPG6)
- net at R601.1, U10.9: now also U8.19 (G26_USB1_D-); no longer U8.37 (LPG2)
- net at Q701.1 (G), R701.1: now also U8.17 (G27_USB1_D+); no longer U8.29 (LPG13)
- net at R24.2, U11.4 (SDA): now also U8.33 (G34__JTAG_ENABLE); no longer U8.6 (LPG9)
- net at R25.2, U11.5 (SCL): now also U8.47 (G36_RMII_MDIO); no longer U8.4 (LPG11)
- net at U8.16 (LPG4): no longer SW2.2
- net at U8.55 (G52_RMII_RST): now also SW2.2
