File: flagship/ossm-flagship.kicad_sch (KiCad schematic)
At the start: 219 parts, among them J1 BUS_IN XT30, J2 MOTOR XT30, J3 EXT_SHUNT XT30, J4 MOTION GH4, J5 COMMS GH6, J6 FAN GH3, J7 THERM GH2, J8 PROBE 1x4 2.54, J9 ESTOP GH3, Q1 IPB042N10N3G, Q2 IPB042N10N3G, Q401 IPB042N10N3G, Q402 IPB042N10N3G, Q403 DMN10H220L, Q404 MMBT3904, Q405 MMBT3904, Q501 IPB042N10N3G, Q701 2N7002, Q702 AO3401A, Q901 2N7002, Q902 2N7002, Q903 2N7002, SW1 HOME (hold: RESET), SW2 PAIR (held at power-on: AP), U1 LTC4364IS-1, U10 74AHCT125, U11 INA228, U2 TPS48111, U3 TLV1805, U4 TLV431, U5 TPS54560B 12V, U6 TPS54560B 5V, U7 TPS54560B 3V3, U8 Stamp-P4, U9 THVD1450

Commit message: flagship: optional accessory breakouts on the spare LP pads (HP-driven); LP rule restated
ACCESSORIES section: PUMP (12 V via 1.25 A polyfuse + PWM on LPG13), EXT PWM
(LPG2, signal only), BUS OUT (+BUS via 2 A 60 V polyfuse), NEOPIXEL OUT chained
after D5 (5 V via 1 A polyfuse), BUTTONS (HOME/PAIR parallel + AUX1/AUX2 on
LPG4/LPG6, 10k pull-ups, 1k, ESD), QWIIC on its own I2C bus (LPG11/LPG9, 2.2k),
GPIO 2x6 (HP UART on LPG14/15, IO1-6 on LPG12/10/8/7/1/0, 220R each).
Connectors are placeholders. LP core still drives QUAD_A/B only; quad jitter
under hammered accessory I/O is Nucleus val-091.18.

Netlist diffed per pin: additions only; the 14 LP pads leave the unconnected
list. ERC: 12 errors, all unused Stamp-P4 pins.
Parts:
- added D1001, D1002: PESD3V3S2UT, Package_TO_SOT_SMD:SOT-23, symbol Device:D_TVS_Dual_AAC
- added F1001: 1.25A 1812L125/33GR, Fuse:Fuse_1812_4532Metric, symbol Device:Polyfuse
- added F1003: 1A 1206L100/24NR, Fuse:Fuse_1206_3216Metric, symbol Device:Polyfuse
- added F1004: 0.2A 1206L020/30NR, Fuse:Fuse_1206_3216Metric, symbol Device:Polyfuse
- added F1005: 2A 2920L200/60GR, Fuse:Fuse_2920_7451Metric, symbol Device:Polyfuse
- added J10: PUMP1 XH3, Connector_JST:JST_XH_B3B-XH-A_1x03_P2.50mm_Vertical, symbol Connector_Generic:Conn_01x03
- added J11: EXT PWM GH2, Connector_JST:JST_GH_SM02B-GHS-TB_1x02-1MP_P1.25mm_Horizontal, symbol Connector_Generic:Conn_01x02
- added J12: NEOPIXEL XH3, Connector_JST:JST_XH_B3B-XH-A_1x03_P2.50mm_Vertical, symbol Connector_Generic:Conn_01x03
- added J13: BUTTONS GH6, Connector_JST:JST_GH_SM06B-GHS-TB_1x06-1MP_P1.25mm_Horizontal, symbol Connector_Generic:Conn_01x06
- added J14: QWIIC SH4, Connector_JST:JST_SH_SM04B-SRSS-TB_1x04-1MP_P1.00mm_Horizontal, symbol Connector_Generic:Conn_01x04
- added J15: GPIO 2x6, Connector_PinHeader_2.54mm:PinHeader_2x06_P2.54mm_Vertical, symbol Connector_Generic:Conn_02x06_Odd_Even
- added J16: BUS OUT XH2, Connector_JST:JST_XH_B2B-XH-A_1x02_P2.50mm_Vertical, symbol Connector_Generic:Conn_01x02
- added R1001, R1002, R1016, R1017, R1018, R1019, R1020, R1021, R1022, R1023: 220R, Resistor_SMD:R_0805_2012Metric, symbol Device:R
- added R1003, R1004: 100k, Resistor_SMD:R_0805_2012Metric, symbol Device:R
- added R1005: 100R, Resistor_SMD:R_0805_2012Metric, symbol Device:R
- added R1006, R1007, R1010, R1011: 1k, Resistor_SMD:R_0805_2012Metric, symbol Device:R
- added R1008, R1009, R1012, R1013: 10k, Resistor_SMD:R_0805_2012Metric, symbol Device:R
- added R1014, R1015: 2.2k, Resistor_SMD:R_0805_2012Metric, symbol Device:R
Connections:
- net +12V: now also F1001.1
- net +3V3_SYS: now also F1004.1, R1008.1, R1009.1, R1012.1, R1013.1
- net +5V: now also F1003.1
- net +BUS: now also F1005.1
- net GND: now also D1001.3 (common), D1002.3 (common), J10.2 (Pin_2), J11.2 (Pin_2), J12.3 (Pin_3), J13.1 (Pin_1), J14.1 (Pin_1), J15.3 (Pin_3), J15.4 (Pin_4), J16.2 (Pin_2), R1003.2, R1004.2
- net at SW1.2, U8.12 (G49_ADC2): now also R1006.1, R1012.2
- net at D5.2 (DOUT): now also R1005.1
- net at U8.1 (LPG15_LPRXD_PCRXD): now also R1017.2
- net at U8.11 (LPG0): now also R1023.2
- net at U8.16 (LPG4): now also R1008.2, R1010.1
- net at U8.18 (LPG6): now also R1009.2, R1011.1
- net at U8.2 (LPG14_LPTXD_PCTXD): now also R1016.2
- net at U8.29 (LPG13): now also R1001.2, R1003.1
- net at U8.3 (LPG12): now also R1018.2
- net at U8.37 (LPG2): now also R1002.2, R1004.1
- net at U8.4 (LPG11): now also J14.3 (Pin_3), R1014.2
- net at U8.5 (LPG10): now also R1019.2
- net at SW2.2, U8.55 (G52_RMII_RST): now also R1007.1, R1013.2
- net at U8.6 (LPG9): now also J14.4 (Pin_4), R1015.2
- net at U8.7 (LPG8): now also R1020.2
- net at U8.8 (LPG7): now also R1021.2
- net at U8.9 (LPG1): now also R1022.2
- new net: J15.12 (Pin_12), R1023.1
- new net: J15.11 (Pin_11), R1022.1
- new net: J15.5 (Pin_5), R1016.1
- new net: J15.8 (Pin_8), R1019.1
- new net: D1002.1 (A1), J13.4 (Pin_4), R1010.2
- new net: D1002.2 (A2), J13.5 (Pin_5), R1011.2
- new net: F1001.2, J10.1 (Pin_1)
- new net: F1005.2, J16.1 (Pin_1)
- new net: J10.3 (Pin_3), R1001.1
- new net: J11.1 (Pin_1), R1002.1
- new net: J15.6 (Pin_6), R1017.1
- new net: J15.10 (Pin_10), R1021.1
- new net: J15.7 (Pin_7), R1018.1
- new net: J15.9 (Pin_9), R1020.1
- new net: D1001.1 (A1), J13.2 (Pin_2), R1006.2
- new net: D1001.2 (A2), J13.3 (Pin_3), R1007.2
- new net: J12.2 (Pin_2), R1005.2
- new net 3V3_ACC: F1004.2, J13.6 (Pin_6), J14.2 (Pin_2), J15.1 (Pin_1), R1014.1, R1015.1
- new net 5V_ACC: F1003.2, J12.1 (Pin_1), J15.2 (Pin_2)
- no-connect marks 7 -> 6
Other:
- note added: "ACCESSORIES"
- note added: "ACCESSORIES (optional; operator 2026-09-23). Simple PWM/on-off loads only; anything with its own logic is a separate Valence device. All on spare LP pads through the HP GPIO matrix: the LP core drives QUAD_A/B only, and firmware must use HP peripherals here (never LP UART/LP I2C, which load the LP bus the emitter uses). PUMP (LPG13): 12 V via a 1.25 A polyfuse + PWM for an off-board MOSFET module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"
