File: flagship/ossm-flagship.kicad_sch (KiCad schematic)
At the start: 277 parts, among them J1 BUS_IN XT30, J10 PUMP1 XH3, J11 EXT PWM GH2, J12 NEOPIXEL XH3, J13 BUTTONS GH6, J14 QWIIC SH4, J15 GPIO 2x6, J16 BUS OUT XH2, J2 MOTOR XT30, J3 EXT_SHUNT XT30, J4 MOTION GH4, J5 COMMS GH6, J6 FAN GH3, J7 THERM GH2, J8 PROBE 1x4 2.54, J9 ESTOP GH3, Q1 IPB042N10N3G, Q2 IPB042N10N3G, Q401 IPB042N10N3G, Q402 IPB042N10N3G, Q403 DMN10H220L, Q404 MMBT3904, Q405 MMBT3904, Q501 IPB042N10N3G, Q701 2N7002, Q702 AO3401A, Q901 2N7002, Q902 2N7002, Q903 2N7002, SW1 HOME (hold: RESET), SW2 PAIR (held at power-on: AP), U1 LTC4364IS-1, U10 74AHCT125, U11 INA228, U12 CH32V003F4U6, U13 AMS1117-3.3, U2 TPS48111, U3 TLV1805, U4 TLV431, U5 TPS54560B 12V, U6 TPS54560B 5V, U8 Stamp-P4, U9 THVD1450

Commit message: flagship: INA228 shunt R2 moved after the motor switch (motor current only); VBUS on MOTOR_V+
Q402 -> SW_OUT -> R2 -> MOTOR_V+ -> J2; JP401 lands on SW_OUT (before R2);
R1 pad 1 joins +BUS; U11 VBUS on MOTOR_V+; monitor channel R1106 moved to +BUS;
POWER MONITOR relocated beside J2 with R24/R25. Kelvin pair as INA_SENSE_P/N
labels (route as a pair on the PCB).

Netlist diffed per pin: exactly the ruled change. ERC identical (53).
Connections:
- net +BUS: now also JP801.2 (B), R1.1, R1106.2, R805.1; no longer R2.1, U11.8 (VBUS)
- net MOTOR_V+: now also R2.1, U11.8 (VBUS); no longer JP401.2 (B), Q402.2 (D), R1106.2
- net INA_SENSE_P: now reaches R2.3, U11.10 (IN+)
- net INA_SENSE_N: now reaches R2.2, U11.9 (IN-)
- new net SW_OUT: JP401.2 (B), Q402.2 (D), R2.4
Other:
- note added: "BOARD MONITOR (operator 2026-09-23): U12 CH32V003F4U6 on the INA228 I2C bus watches VIN_RAW, +BUS, +12V, +5V, +3V3_ACC, +5V_SYS, CLAMP_MON and SHUNT_TEMP (VIN_RAW vs +BUS = the input-stage check; the INA228 covers motor voltage). FAULT_N (open-drain, 1k) joins the motor-switch EN wired-OR: it can cut motor power, never enable it. CLAMP_TRIM (PWM -> 10k -> 1u -> 47k into U3 +IN; 10k pull-down at t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"
- note added: "SENSING (record sections 10, 12). U11 INA228 on R2 AFTER the motor switch: motor current only (sensorless homing); VBUS on MOTOR_V+ shows motor power; JP401 lands before R2. Motoring reads positive, regen negative. Route INA_SENSE_P/N as a tight pair, INA beside the shunt, away from switch nodes. 1 mOhm: 10 mV at 10 A in the +-163.84 mV range. Die temperature = board temperature. A0/A1 = GND (0x4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"
- note removed: "BOARD MONITOR (operator 2026-09-23): U12 CH32V003F4U6 on the INA228 I2C bus watches VIN_RAW, MOTOR_V+, +12V, +5V, +3V3_ACC, +5V_SYS, CLAMP_MON and SHUNT_TEMP. FAULT_N (open-drain, 1k) joins the motor-switch EN wired-OR: it can cut motor power, never enable it. CLAMP_TRIM (PWM -> 10k -> 1u -> 47k into U3 +IN; 10k pull-down at the pin; R502 12.1k) can only LOWER the regen threshold: duty 0 = 44.5 V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"
- note removed: "SENSING (record sections 10, 12). U11 INA228 on the R2 Kelvin taps (Input sheet): route INA_SENSE_P/N as a tight pair, INA beside the shunt, away from switch nodes. 1 mOhm: 10 mV at 10 A in the +-163.84 mV range. Die temperature = board temperature. A0/A1 = GND (0x40). INA_ALERT_N (open drain) is also the motor-switch EN: over-current / power / temperature limits cut the motor with no MCU. R24/R2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"
- moved on the sheet: C13, D401, R2, R24, R25, U11

Commit message: flagship: pump eFuse (TPS259541, 2.5 A) + BUS OUT removed; layout: bucks stacked, OVP trip inside MOTOR SWITCH, thermistor moved
Electrical: F1001 polyfuse -> U14 TPS259541DSGR (R_ILM 806R = 2.52 A, EN
64.9k/10k = 9.0 V, dVdt 3.3 nF, FLT -> U12 PC0); J16/F1005 BUS OUT deleted.
New local symbol flagship:TPS259541DSGR (pinout from TI SLVSE57C).
Layout (connectivity-neutral): BUCK RAILS 12 V / 5 V / LDO stacked; bus OVP
trip (D402/R413/R414/Q405) moved inside MOTOR SWITCH; TH501/R512 moved beside
the CLAMP_MON divider.

Netlist diffed per pin: only the eFuse/BUS OUT changes; the layout passes are
zero-change. ERC: 11 errors (unused Stamp-P4 pins, unchanged); +9 pin_to_pin
warnings from U14's unspecified pin types (house convention).
Parts:
- removed F1001: 1.25A 1812L125/33GR, Fuse:Fuse_1812_4532Metric, symbol Device:Polyfuse
- removed F1005: 2A 2920L200/60GR, Fuse:Fuse_2920_7451Metric, symbol Device:Polyfuse
- removed J16: BUS OUT XH2, Connector_JST:JST_XH_B2B-XH-A_1x02_P2.50mm_Vertical, symbol Connector_Generic:Conn_01x02
- added C1201: 3.3n, Capacitor_SMD:C_0805_2012Metric, symbol Device:C
- added C1202: 1u 25V, Capacitor_SMD:C_0805_2012Metric, symbol Device:C
- added R1201: 806R, Resistor_SMD:R_0805_2012Metric, symbol Device:R
- added R1202: 64.9k, Resistor_SMD:R_0805_2012Metric, symbol Device:R
- added R1203, R1204: 10k, Resistor_SMD:R_0805_2012Metric, symbol Device:R
- added U14: TPS259541DSGR, Package_SON:Texas_DSG0008A_WSON-8-1EP_2x2mm_P0.5mm_EP0.9x1.6mm, symbol flagship:TPS259541DSGR
Connections:
- net +12V: now also C1202.1, R1202.1, U14.3 (IN), U14.4 (IN)
- net +3V3_SYS: now also R1204.1
- net GND: now also C1201.1, C1202.2, R1201.1, U14.8 (GND), U14.9 (EP)
- net at J10.1 (Pin_1): now also U14.5 (OUT)
- net PUMP_FLT: now reaches U12.7 (PC0)
- net PUMP_FLT: now also R1204.2, U14.6 (~{FLT})
- new net: C1201.2, R1203.2, U14.1 (dVdt), U14.2 (EN/UVLO)
- new net: R1201.2, U14.7 (ILM)
- new net: R1202.2, R1203.1
- no-connect marks 10 -> 9
Other:
- note added: "ACCESSORIES (optional; operator 2026-09-23). Simple PWM/on-off loads only; anything with its own logic is a separate Valence device. All on spare LP pads through the HP GPIO matrix: the LP core drives QUAD_A/B only, and firmware must use HP peripherals here (never LP UART/LP I2C, which load the LP bus the emitter uses). PUMP (LPG13): 12 V through U14 TPS259541 eFuse (2.5 A limit, 13.7 V output cl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"
- note removed: "ACCESSORIES (optional; operator 2026-09-23). Simple PWM/on-off loads only; anything with its own logic is a separate Valence device. All on spare LP pads through the HP GPIO matrix: the LP core drives QUAD_A/B only, and firmware must use HP peripherals here (never LP UART/LP I2C, which load the LP bus the emitter uses). PUMP (LPG13): 12 V via a 1.25 A polyfuse + PWM for an off-board MOSFET module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"
- moved on the sheet: C1301, C1302, C201, C202, C203, C204, C205, C206, C207, C208, C209, C210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
